File: Tilty Hardware/Board Files/Dual Motor Driver/V0.1.0/Eagle PCB Files/Dual Motor Driver.brd (EAGLE design)
At the start: 50.8 x 50.8 mm, 36 parts, among them J1 AVR_SPI_PRG_6PTH, Q1 16MHz, U1 ATMEGA32U4QFN2, U2 L298_BRIDGE_DRIVER, U5 VOLTAGE-REGULATOR

Commit message: Dual motor driver pcb work
Parts:
- removed JP10, JP9: M12LOCK, SparkFun-Connectors:1X12_LOCK
- added S1: SWITCH-MOMENTARY-2SMD, SparkFun-Electromechanical:TACTILE_SWITCH_SMD
Connections:
- removed net DIO0/RX: U1.20
- removed net DIO1/TX: U1.21
- removed net DIO10: U1.30
- removed net DIO12: U1.26
- removed net DIO4: U1.25
- removed net DIO5: U1.31
- removed net DIO6: U1.27
- removed net DIO7: U1.1
- removed net DIO8: U1.28
- removed net DIO9: U1.29
- new net ENC1A: JP6.P$3, U1.1
- new net ENC1B: JP6.P$4, U1.20
- new net ENC2A: JP5.P$4, U1.26
- new net ENC2B: JP5.P$3, U1.21
- new net M1+: U1.25, U2.7
- new net M1-: U1.28, U2.9
- new net M2+: U1.31, U2.13
- new net M2-: U1.27, U2.15
- new net PWM1: U1.29, U2.8
- new net PWM2: U1.30, U2.14
- net +5V: now also JP5.P$1, JP6.P$6
- net GND: now also JP5.P$2, JP6.P$5, S1.1
- net |HWB: now also S1.3
Changed lines of the file:
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@@
 <setting verticaltext="up"/>
 </settings>
-<grid distance="0.01" unitdist="inch" unit="inch" style="lines" multiple="1" display="yes" altdistance="0.005" altunitdist="inch" altunit="inch"/>
+<grid distance="0.05" unitdist="inch" unit="inch" style="lines" multiple="1" display="yes" altdistance="0.005" altunitdist="inch" altunit="inch"/>
 <layers>
 <layer number="1" name="Top" color="4" fill="1" visible="yes" active="yes"/>
@@
 <element name="C2" library="resistor" package="C0603" value="22pF" x="33.782" y="28.956" smashed="yes"/>
 <element name="C8" library="resistor" package="C0603" value="22pF" x="33.02" y="36.576" smashed="yes" rot="R180"/>
-<element name="JP10" library="SparkFun-Connectors" package="1X12_LOCK" value="M12LOCK" x="48.514" y="19.304" rot="R90"/>
 <element name="R2" library="resistor" package="R0603" value="10K" x="21.844" y="38.1" rot="R180"/>
-<element name="JP9" library="SparkFun-Connectors" package="1X12_LOCK" value="M12LOCK" x="3.556" y="19.05" rot="R90"/>
+<element name="S1" library="SparkFun-Electromechanical" package="TACTILE_SWITCH_SMD" value="SWITCH-MOMENTARY-2SMD" x="18.542" y="44.196" rot="R270"/>
 </elements>
 <signals>
@@
 <wire x1="37.465" y1="10.922" x2="37.465" y2="9.222" width="0.508" layer="1"/>
 <wire x1="37.465" y1="16.891" x2="37.465" y2="18.591" width="0.508" layer="1"/>
-<wire x1="37.465" y1="18.591" x2="38.608" y2="21.59" width="0" layer="19" extent="1-1"/>
-<wire x1="32.385" y1="9.525" x2="37.465" y2="9.222" width="0" layer="19" extent="1-1"/>
-<wire x1="32.385" y1="20.955" x2="37.465" y2="18.591" width="0" layer="19" extent="1-1"/>
-<wire x1="32.932" y1="28.956" x2="32.385" y2="20.955" width="0" layer="19" extent="1-1"/>
-<wire x1="28.8" y1="32.274" x2="32.932" y2="28.956" width="0" layer="19" extent="1-1"/>
-<wire x1="27.9" y1="36.674" x2="28.8" y2="32.274" width="0" layer="19" extent="1-1"/>
-<wire x1="28.448" y1="42.584" x2="27.9" y2="36.674" width="0" layer="19" extent="1-1"/>
+<contactref element="JP5" pad="P$2"/>
+<contactref element="JP6" pad="P$5"/>
+<contactref element="S1" pad="1"/>
 <wire x1="22.86" y1="42.584" x2="28.448" y2="42.584" width="0" layer="19" extent="1-1"/>
+<wire x1="20.447" y1="46.736" x2="22.86" y2="42.584" width="0" layer="19" extent="1-1"/>
+<wire x1="27.9" y1="36.674" x2="28.448" y2="42.584" width="0" layer="19" extent="1-1"/>
+<wire x1="28.8" y1="32.274" x2="27.9" y2="36.674" width="0" layer="19" extent="1-1"/>
+<wire x1="32.932" y1="28.956" x2="28.8" y2="32.274" width="0" layer="19" extent="1-1"/>
 <wire x1="33.87" y1="36.576" x2="27.9" y2="36.674" width="0" layer="19" extent="1-1"/>
 <wire x1="22" y1="35.274" x2="27.9" y2="36.674" width="0" layer="19" extent="1-1"/>
@@
 <wire x1="13.843" y1="18.591" x2="15.074" y2="21.59" width="0" layer="19" extent="1-1"/>
 <wire x1="18.923" y1="20.955" x2="15.074" y2="21.59" width="0" layer="19" extent="1-1"/>
+<wire x1="32.385" y1="20.955" x2="32.932" y2="28.956" width="0" layer="19" extent="1-1"/>
+<wire x1="37.465" y1="18.591" x2="32.385" y2="20.955" width="0" layer="19" extent="1-1"/>
+<wire x1="38.608" y1="21.59" x2="37.465" y2="18.591" width="0" layer="19" extent="1-1"/>
+<wire x1="32.385" y1="9.525" x2="37.465" y2="9.222" width="0" layer="19" extent="1-1"/>
+<wire x1="45.373" y1="10.898" x2="37.465" y2="10.922" width="0" layer="19" extent="1-16"/>
+<wire x1="5.427" y1="10.644" x2="13.843" y2="10.922" width="0" layer="19" extent="1-16"/>
 <wire x1="23.764" y1="3.556" x2="32.385" y2="9.525" width="0" layer="19" extent="1-1"/>
 </signal>
@@
 <contactref element="U5" pad="P$1"/>
 <contactref element="R2" pad="2"/>
+<contactref element="JP5" pad="P$1"/>
+<contactref element="JP6" pad="P$6"/>
 <wire x1="30.226" y1="43.304" x2="30.988" y2="47.664" width="0" layer="19" extent="1-1"/>
 <wire x1="27.4" y1="36.674" x2="30.226" y2="43.304" width="0" layer="19" extent="1-1"/>
@@
 <wire x1="31.076" y1="28.702" x2="28.8" y2="31.774" width="0" layer="19" extent="1-1"/>
 <wire x1="22" y1="35.774" x2="22" y2="30.774" width="0" layer="19" extent="1-1"/>
+<wire x1="20.994" y1="38.1" x2="22" y2="35.774" width="0" layer="19" extent="1-1"/>
 <wire x1="38.608" y1="26.67" x2="31.076" y2="28.702" width="0" layer="19" extent="1-1"/>
 <wire x1="18.923" y1="19.685" x2="20.828" y2="29.122" width="0" layer="19" extent="1-1"/>
 <wire x1="13.374" y1="21.59" x2="18.923" y2="19.685" width="0" layer="19" extent="1-1"/>
 <wire x1="13.237" y1="23.113" x2="13.374" y2="21.59" width="0" layer="19" extent="1-1"/>
-<wire x1="20.994" y1="38.1" x2="13.374" y2="21.59" width="0" layer="19" extent="1-1"/>
+<wire x1="5.427" y1="11.644" x2="13.374" y2="21.59" width="0" layer="19" extent="1-1"/>
+<wire x1="45.373" y1="11.898" x2="38.608" y2="26.67" width="0" layer="19" extent="1-1"/>
 </signal>
 <signal name="USB_D-">
@@
 <contactref element="R1" pad="1"/>
 <contactref element="U1" pad="13"/>
-<wire x1="29.376" y1="28.702" x2="36.068" y2="21.59" width="0" layer="19" extent="1-1"/>
-<wire x1="28.8" y1="31.274" x2="29.376" y2="28.702" width="0" layer="19" extent="1-1"/>
+<wire x1="29.376" y1="28.702" x2="28.8" y2="31.274" width="0" layer="19" extent="1-1"/>
+<wire x1="36.068" y1="21.59" x2="29.376" y2="28.702" width="0" layer="19" extent="1-1"/>
 </signal>
 <signal name="SCK">
@@
 <contactref element="U1" pad="36"/>
 </signal>
-<signal name="DIO0/RX">
-<contactref element="U1" pad="20"/>
-</signal>
-<signal name="DIO1/TX">
-<contactref element="U1" pad="21"/>
-</signal>
-<signal name="DIO4">
-<contactref element="U1" pad="25"/>
-</signal>
-<signal name="DIO5">
-<contactref element="U1" pad="31"/>
-</signal>
-<signal name="DIO6">
-<contactref element="U1" pad="27"/>
-</signal>
-<signal name="DIO7">
-<contactref element="U1" pad="1"/>
-</signal>
-<signal name="DIO8">
-<contactref element="U1" pad="28"/>
-</signal>
-<signal name="DIO9">
-<contactref element="U1" pad="29"/>
-</signal>
-<signal name="DIO10">
-<contactref element="U1" pad="30"/>
-</signal>
 <signal name="DIO11">
 <contactref element="U1" pad="12"/>
-</signal>
-<signal name="DIO12">
-<contactref element="U1" pad="26"/>
 </signal>
 <signal name="DIO13">
@@
 <contactref element="U1" pad="33"/>
 <contactref element="R2" pad="1"/>
-<wire x1="22.694" y1="38.1" x2="22.9" y2="36.674" width="0" layer="19" extent="1-1"/>
+<contactref element="S1" pad="3"/>
+<wire x1="22.694" y1="38.1" x2="16.637" y2="46.736" width="0" layer="19" extent="1-1"/>
+<wire x1="22.9" y1="36.674" x2="22.694" y2="38.1" width="0" layer="19" extent="1-1"/>
+</signal>
+<signal name="ENC1B">
+<contactref element="JP6" pad="P$4"/>
+<contactref element="U1" pad="20"/>
+<wire x1="45.373" y1="9.898" x2="28.8" y2="34.774" width="0" layer="19" extent="1-1"/>
+</signal>
+<signal name="ENC1A">
+<contactref element="JP6" pad="P$3"/>
+<contactref element="U1" pad="1"/>
+<wire x1="22.9" y1="29.874" x2="45.373" y2="8.898" width="0" layer="19" extent="1-1"/>
+</signal>
+<signal name="ENC2B">
+<contactref element="JP5" pad="P$3"/>
+<contactref element="U1" pad="21"/>
+<wire x1="5.427" y1="9.644" x2="28.8" y2="35.274" width="0" layer="19" extent="1-1"/>
+</signal>
+<signal name="ENC2A">
+<contactref element="JP5" pad="P$4"/>
+<contactref element="U1" pad="26"/>
+<wire x1="5.427" y1="8.644" x2="26.4" y2="36.674" width="0" layer="19" extent="1-1"/>
+</signal>
+<signal name="M1+">
+<contactref element="U2" pad="7"/>
+<contactref element="U1" pad="25"/>
+<wire x1="32.385" y1="17.145" x2="26.9" y2="36.674" width="0" layer="19" extent="1-1"/>
+</signal>
+<signal name="M1-">
+<contactref element="U2" pad="9"/>
+<contactref element="U1" pad="28"/>
+<wire x1="32.385" y1="19.685" x2="25.4" y2="36.674" width="0" layer="19" extent="1-1"/>
+</signal>
+<signal name="M2-">
+<contactref element="U2" pad="15"/>
+<contactref element="U1" pad="27"/>
+<wire x1="18.923" y1="15.875" x2="25.9" y2="36.674" width="0" layer="19" extent="1-1"/>
+</signal>
+<signal name="M2+">
+<contactref element="U2" pad="13"/>
+<contactref element="U1" pad="31"/>
+<wire x1="18.923" y1="18.415" x2="23.9" y2="36.674" width="0" layer="19" extent="1-1"/>
+</signal>
+<signal name="PWM2">
+<contactref element="U2" pad="14"/>
+<contactref element="U1" pad="30"/>
+<wire x1="18.923" y1="17.145" x2="24.4" y2="36.674" width="0" layer="19" extent="1-1"/>
+</signal>
+<signal name="PWM1">
+<contactref element="U2" pad="8"/>
+<contactref element="U1" pad="29"/>
+<wire x1="32.385" y1="18.415" x2="24.9" y2="36.674" width="0" layer="19" extent="1-1"/>
 </signal>
 </signals>
