File: Tilty Hardware/Board Files/Tilty Duo:Quad/V0.2.4/Eagle PCB Files/TiltyDuo.sch (EAGLE design)
At the start: 45 parts, among them U1 TEENSY_3.0_OUTER-PINS28-DIP_S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, U2 HC-09_BREAKOUT, U3 MPL3115A2LGA8, U4 LM2931, U5 MPU-6050, U6 HMC5883LSMD, U7 SPI_FLASH-X25XXSMD

Commit message: Minor part # changes
alternative part #'s for some Tilty Duo/Quad components
Parts:
- U1: PART#3 (none) -> ED3052-5-ND
Changed lines of the file:
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@@
 <attribute name="PART#" value="AE10004-ND"/>
 <attribute name="PART#2" value="A28-LC-TR-R"/>
+<attribute name="PART#3" value="ED3052-5-ND"/>
 </part>
 <part name="JP1" library="pinhead" deviceset="PINHD-1X8" device="1X08_NO_SILK_LOCK"/>
@@
 <attribute name="PART#" x="187.96" y="45.72" size="1.778" layer="96" display="off"/>
 <attribute name="PART#2" x="187.96" y="45.72" size="1.778" layer="96" display="off"/>
+<attribute name="PART#3" x="187.96" y="45.72" size="1.778" layer="96" display="off"/>
 </instance>
 <instance part="JP1" gate="A" x="139.7" y="53.34" rot="R180"/>
