File: Tilty Hardware/Board Files/Tilty Omni/V0.1.0/Eagle PCB Files/TiltyOmni.sch (EAGLE design)
At the start: 38 parts, among them U1 TEENSY_3.0_ALLPINS, U2 HC-09_BREAKOUT, U4 LM2931, U5 MPU-6050, U7 SPI_FLASH-X25XXSMD

Commit message: More work on the Tilty Omni
Connections:
- removed net SCL: R1.1, U5.SCL
- removed net SDA: R2.1, U5.SDA
- removed net TEENSY_3V3: C2.2, U5.VDD
- net +3V3: now also C2.2, U5.VDD
- net 3V_SCL: now also R1.1, U5.SCL
- net 3V_SDA: now also R2.1, U5.SDA
Changed lines of the file:
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@@
 <part name="JP6" library="SparkFun-Connectors" deviceset="M20" device=""/>
 <part name="JP7" library="SparkFun-Connectors" deviceset="M20" device=""/>
+<part name="+3V7" library="supply1" deviceset="+3V3" device=""/>
 </parts>
 <sheets>
@@
 <instance part="JP6" gate="G$1" x="266.7" y="48.26"/>
 <instance part="JP7" gate="G$1" x="284.48" y="48.26"/>
+<instance part="+3V7" gate="G$1" x="20.32" y="119.38"/>
 </instances>
 <busses>
@@
 </segment>
 </net>
-<net name="SCL" class="4">
-<segment>
-<pinref part="U5" gate="G$1" pin="SCL"/>
-<pinref part="R1" gate="G$1" pin="1"/>
-<wire x1="66.04" y1="109.22" x2="83.82" y2="109.22" width="0.1524" layer="91"/>
-<label x="66.04" y="109.22" size="1.524" layer="95"/>
-</segment>
-</net>
-<net name="SDA" class="4">
-<segment>
-<pinref part="U5" gate="G$1" pin="SDA"/>
-<pinref part="R2" gate="G$1" pin="1"/>
-<wire x1="66.04" y1="104.14" x2="78.74" y2="104.14" width="0.1524" layer="91"/>
-<label x="66.04" y="104.14" size="1.524" layer="95"/>
-</segment>
-</net>
 <net name="N$1" class="0">
 <segment>
@@
 <segment>
 <pinref part="MPU_INT" gate="1" pin="1"/>
-<wire x1="7.62" y1="109.22" x2="7.62" y2="116.84" width="0.1524" layer="91"/>
-<wire x1="7.62" y1="116.84" x2="20.32" y2="116.84" width="0.1524" layer="91"/>
-<label x="10.16" y="116.84" size="1.778" layer="95"/>
+<wire x1="7.62" y1="109.22" x2="7.62" y2="127" width="0.1524" layer="91"/>
+<wire x1="7.62" y1="127" x2="20.32" y2="127" width="0.1524" layer="91"/>
+<label x="10.16" y="127" size="1.778" layer="95"/>
 </segment>
 </net>
@@
 </segment>
 </net>
-<net name="TEENSY_3V3" class="3">
-<segment>
-<pinref part="U5" gate="G$1" pin="VDD"/>
-<wire x1="30.48" y1="111.76" x2="27.94" y2="111.76" width="0.1524" layer="91"/>
-<pinref part="C2" gate="G$1" pin="2"/>
-<wire x1="27.94" y1="111.76" x2="11.43" y2="111.76" width="0.1524" layer="91"/>
-<wire x1="27.94" y1="116.84" x2="27.94" y2="111.76" width="0.1524" layer="91"/>
-<junction x="27.94" y="111.76"/>
-<label x="11.43" y="111.76" size="1.778" layer="95"/>
-</segment>
-</net>
 <net name="5V" class="0">
 <segment>
@@
 <label x="241.3" y="17.78" size="1.778" layer="95"/>
 </segment>
+<segment>
+<pinref part="U5" gate="G$1" pin="SCL"/>
+<pinref part="R1" gate="G$1" pin="1"/>
+<wire x1="66.04" y1="109.22" x2="83.82" y2="109.22" width="0.1524" layer="91"/>
+<label x="66.04" y="109.22" size="1.524" layer="95"/>
+</segment>
 </net>
 <net name="3V_SDA" class="0">
@@
 <wire x1="231.14" y1="15.24" x2="251.46" y2="15.24" width="0.1524" layer="91"/>
 <label x="241.3" y="15.24" size="1.778" layer="95"/>
+</segment>
+<segment>
+<pinref part="U5" gate="G$1" pin="SDA"/>
+<pinref part="R2" gate="G$1" pin="1"/>
+<wire x1="66.04" y1="104.14" x2="78.74" y2="104.14" width="0.1524" layer="91"/>
+<label x="66.04" y="104.14" size="1.524" layer="95"/>
 </segment>
 </net>
@@
 <pinref part="+3V6" gate="G$1" pin="+3V3"/>
 </segment>
-</net>
+<segment>
+<pinref part="U5" gate="G$1" pin="VDD"/>
+<wire x1="30.48" y1="111.76" x2="27.94" y2="111.76" width="0.1524" layer="91"/>
+<pinref part="C2" gate="G$1" pin="2"/>
+<wire x1="27.94" y1="116.84" x2="27.94" y2="111.76" width="0.1524" layer="91"/>
+<pinref part="+3V7" gate="G$1" pin="+3V3"/>
+<wire x1="27.94" y1="111.76" x2="20.32" y2="111.76" width="0.1524" layer="91"/>
+<wire x1="20.32" y1="111.76" x2="20.32" y2="116.84" width="0.1524" layer="91"/>
+<junction x="27.94" y="111.76"/>
+</segment>
+</net>

Commit message: Tilty Omni updates, updated things to do
Parts:
- C5: value 0.1uF -> 4.7uF
Connections:
- removed net 5V: D2.A
- removed net N$10: U1.5/PWM
- removed net VBATT: C4.1, JP5.P$1, SJ4.1, U4.VIN
- new net 24: U1.24
- new net 25: U1.25
- new net 26: U1.26
- new net 27: U1.27
- new net 28: U1.28
- new net 29: U1.29
- new net 30: U1.30
- new net 31: U1.31
- new net 32: U1.32
- new net 33: U1.33
- new net A10: U1.A10
- new net A11: U1.A11
- new net A12: U1.A12
- new net A13: U1.A13
- net +5V: now also D2.A
- net GND: now also JP5.2; no longer JP5.P$2
- net IMU_INT: now also U1.5/PWM
- net VCC: now also C4.1, JP5.1, SJ4.1, U4.VIN
Other:
- moved on the sheet: D2, R5, R6, SJ4

Commit message: Tilty PCB work
Parts:
- U1: value TEENSY_3.0_ALLPINS -> TEENSY_3.0_ALLPINSTEENSY_3.0_ALLPINS-SMD; device Teensy3.0:TEENSY_3.0_ALLPINS -> Teensy3.0:TEENSY_3.0_ALLPINSTEENSY_3.0_ALLPINS-SMD
Changed lines of the file:
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@@
 </part>
 <part name="GND23" library="supply1" deviceset="GND" device=""/>
-<part name="U1" library="Teensy3.0" deviceset="TEENSY_3.0_ALLPINS" device="" value="TEENSY_3.0_ALLPINS"/>
+<part name="U1" library="Teensy3.0" deviceset="TEENSY_3.0_ALLPINS" device="TEENSY_3.0_ALLPINS-SMD" value="TEENSY_3.0_ALLPINSTEENSY_3.0_ALLPINS-SMD"/>
 <part name="GND6" library="supply1" deviceset="GND" device=""/>
 <part name="GND8" library="supply1" deviceset="GND" device=""/>

Commit message: LOTS of work on the Tilty Omni
Parts:
- MPU_INT: value SOLDERJUMPERNO -> SOLDERJUMPERTRACE; device SparkFun-Passives:SOLDERJUMPERNO -> SparkFun-Passives:SOLDERJUMPERTRACE
Connections:
- removed net 33: U1.33
- removed net A13: U1.A13
- removed net AUX_SCL: JP3.7
- removed net AUX_SDA: JP3.6
- removed net MPU_INT: MPU_INT.1
- new net 14/A0: JP3.4, U1.14/A0
- new net 15/A1: JP3.3, U1.15/A1/CS4
- new net 5/PWM: JP1.7, JP6.14, U1.5/PWM
- new net 6/PWM: JP6.13, U1.6/PWM
- new net N$30: JP7.1
- new net N$31: JP7.2
- new net N$32: JP7.3
- new net N$33: JP7.4
- new net N$34: JP7.5
- new net N$35: JP7.6
- new net N$36: JP7.7
- new net N$37: JP7.8
- new net N$38: JP7.9
- new net N$39: JP7.10
- new net N$40: JP7.11
- new net N$41: JP7.12
- new net N$42: JP7.13
- new net N$43: JP7.14
- new net N$44: JP7.15
- new net N$45: JP7.16
- new net N$46: JP7.17
- new net N$47: JP7.18
- new net N$48: JP7.19
- new net N$49: JP7.20
- net 10/TX2: now also JP6.9
- net 24: now also JP6.5
- net 25: now also JP6.4
- net 26: now also JP6.3
- net 27: now also JP6.2
- net 28: now also JP6.1; no longer U1.28
- net 4/PWM: now also JP6.15
- net 7/RX3: now also JP6.12
- net 8/TX3: now also JP6.11
- net 9/RX2: now also JP6.10
- net AUXCL: now also JP3.7
- net AUXDA: now also JP3.6
- net BATT_SENSE: now also U1.A13; no longer JP3.4, U1.14/A0
- net BLUETOOTH_RX: now also JP6.19
- net BLUETOOTH_TX: now also JP6.18
- net BT_CMD: now also U1.28; no longer JP3.3, U1.15/A1/CS4
- net GND: now also JP6.20
- net IMU_INT: now also MPU_INT.1, U1.33; no longer JP1.7, U1.5/PWM
- net MEMORY_CS: no longer U1.6/PWM
- net MISO: now also JP6.7
- net MOSI: now also JP6.8
- net SCK: now also JP6.6
- net SERVO_1: now also JP6.17
- net SERVO_2: now also JP6.16
Other:
- moved on the sheet: JP6, JP7

Commit message: Lots more Tilty Omni work!
Connections:
- net N$48 renamed AGND
- removed net 28: JP6.1
- removed net N$30: JP7.1
- removed net N$31: JP7.2
- removed net N$32: JP7.3
- removed net N$33: JP7.4
- removed net N$34: JP7.5
- removed net N$35: JP7.6
- removed net N$36: JP7.7
- removed net N$37: JP7.8
- removed net N$38: JP7.9
- removed net N$39: JP7.10
- removed net N$40: JP7.11
- removed net N$41: JP7.12
- removed net N$42: JP7.13
- removed net N$43: JP7.14
- removed net N$44: JP7.15
- removed net N$45: JP7.16
- removed net N$46: JP7.17
- removed net N$47: JP7.18
- removed net N$49: JP7.20
- net +3V3: now also JP7.18
- net +5V: now also JP7.20
- net 14/A0: now also JP7.8
- net 15/A1: now also JP7.9
- net 20/A6: now also JP7.14
- net 21/A7: now also JP7.15
- net 27: no longer U1.27
- net 29: now also JP7.1
- net 30: now also JP7.2
- net 31: now also JP7.3
- net 32: now also JP7.4
- net 3V_SCL: now also JP7.13
- net 3V_SDA: now also JP7.12
- net 5V_SCL: now also JP7.10, JP7.11
- net 6/PWM: now also JP1.8
- net A10: now also JP7.7
- net A11: now also JP7.6
- net A12: now also JP7.5
- net BLUETOOTH_RX: now also U2.UART_TX
- net BLUETOOTH_TX: now also U2.UART_RX
- net MEMORY_CS: now also JP6.1, U1.27; no longer JP1.8
- net RX1: no longer U2.UART_TX
- net SERVO_3: now also JP7.16
- net SERVO_4: now also JP7.17
- net TX1: no longer U2.UART_RX
