File: Tilty Hardware/Board Files/Tilty Omni/V0.1.0/Eagle PCB Files/TiltyOmni.brd (EAGLE design)
At the start: 38.1 x 50.8 mm, 40 parts, among them U2 HC-09_BREAKOUT, U4 LM2931, U5 MPU-6050, U7 SPI_FLASH-X25XXSMD

Commit message: Serious work on the Tilty Omni has begun!
Parts:
- removed SJ2, SJ3: (no value), SparkFun-Passives:SJ_3
- removed U$1: TEENSY_3.0_ALLPINSTEENSY_3.0_ALLPINS-SMD, Teensy3.0:TEENSY_3.0_ALLPINS-SMD
- added U1: TEENSY_3.0_ALLPINS, Teensy3.0:TEENSY_3.0_ALLPINS
- JP1, JP2: value (none) -> 8-PIN_HEADER; device pinhead:1X08_NO_SS_LOCKING -> My Parts:8-PIN_RECEPTACLE_LOCK_NO-SS
- JP3: value (none) -> 8-PIN_HEADER; device pinhead:2X03_NO_SS_LOCK -> My Parts:8-PIN_RECEPTACLE_LOCK_NO-SS
- JP4: value 2-POS_SMD_TERM_BLOCK -> 8-PIN_HEADER; device My Parts:2-POS_SMD_TERMINAL_BLOCK -> My Parts:8-PIN_RECEPTACLE_LOCK_NO-SS
- JP5: value (none) -> 2-POS_SMD_TERM_BLOCK; device pinhead:1X08_NO_SS_LOCKING -> My Parts:2-POS_SMD_TERMINAL_BLOCK
- JP6: value (none) -> M20; device pinhead:1X08_NO_SS_LOCKING -> SparkFun-Connectors:1X20
- JP7: value (none) -> M20; device pinhead:2X03_NO_SS_LOCK -> SparkFun-Connectors:1X20
- moved SJ5 119.2 mm to (-58.4, 80.0), turned to 0 degrees
- moved R3 113.0 mm to (-63.5, 69.8), flipped to the top, turned to 0 degrees
- moved R7 111.9 mm to (-58.4, 69.8), flipped to the top, turned to 0 degrees
- moved R5 109.1 mm to (-73.7, 69.8), flipped to the top, turned to 0 degrees
- moved D3 108.4 mm to (-72.4, 40.6)
- moved R6 107.8 mm to (-68.6, 69.8), flipped to the top, turned to 0 degrees
- moved C9 106.1 mm to (-57.1, 76.2), flipped to the top, turned to 0 degrees
- moved C11 95.4 mm to (-63.5, 76.2), flipped to the top, turned to 0 degrees
- moved C13 93.4 mm to (-69.8, 76.2), flipped to the top, turned to 0 degrees
- moved SJ4 87.1 mm to (-31.8, 81.3), turned to 0 degrees
- moved JP9 86.2 mm to (-19.1, 81.3), turned to 0 degrees
- moved R4 86.1 mm to (-15.2, 76.2), flipped to the top, turned to 0 degrees
- moved R8 85.9 mm to (-19.1, 76.2), flipped to the top, turned to 0 degrees
- moved D2 84.1 mm to (-19.1, 69.8)
- moved D1 82.4 mm to (-25.4, 69.8)
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Connections:
- removed net 3.3V: U$1.3.3V, U$1.3.3V1, U$1.3.3V2
- removed net CS: U7.1
- removed net I/O1: JP3.6
- removed net I/O2: JP3.5
- removed net I/O3: JP7.5
- removed net I/O4: JP7.6
- removed net POW_I/O1: JP3.3, JP3.4, SJ2.2
- removed net POW_I/O2: JP7.3, JP7.4, SJ3.2
- removed net VIN: U$1.VIN
- new net +3V3: C11.2, C13.2, C9.1, D5.3, JP1.P$1, R1.2, R2.2, U1.3.3V, U1.3.3V1, U1.3.3V2, U2.P$11, U2.P$12, U5.8, U7.3, U7.7, U7.8
- new net +5V: C5.1, D4.1, JP4.P$1, JP9.4, U4.P$3
- new net 10/TX2: JP2.P$4, U1.10
- new net 20/A6: JP4.P$6, U1.20/A6
- new net 21/A7: JP4.P$5, U1.21/A7
- new net 3V_SCL: JP4.P$7, U1.19/A5
- new net 3V_SDA: JP4.P$8, U1.18/A4
- new net 4/PWM: JP1.P$6, U1.4
- new net 5V_SCL: JP3.P$2, U1.16/A2
- new net 5V_SDA: JP3.P$1, U1.17/A3
- new net 7/RX3: JP2.P$1, U1.7
- new net 8/TX3: JP2.P$2, U1.8
- new net 9/RX2: JP2.P$3, U1.9
- new net AUX_SCL: JP3.P$7
- new net AUX_SDA: JP3.P$6
- new net BLUETOOTH_RX: JP1.P$2, U1.0
- new net BLUETOOTH_TX: JP1.P$3, U1.1
- new net IMU_INT: JP1.P$7
- new net MEMORY_CS: JP1.P$8, U1.6, U7.1
- new net N$10: U1.5
- new net N$4: D4.3, U1.VIN
- new net SERVO_1: JP1.P$4, U1.2
- new net SERVO_2: JP1.P$5, U1.3
- new net SERVO_3: JP4.P$4, U1.22/A8
- new net SERVO_4: JP4.P$3, U1.23/A9
- new net VCC: JP2.P$7
- net 5V: no longer C5.1, JP9.4, SJ2.1, SJ3.1, U4.P$3
- net AGND: now also U1.AGND; no longer U$1.AGND
- net AREF: now also U1.AREF; no longer U$1.AREF
- net BATT_SENSE: now also JP3.P$4, U1.14/A0
- net BT_CMD: now also JP3.P$3, U1.15/A1
- net GND: now also JP2.P$8, JP3.P$8, JP4.P$2, JP5.P$4, U1.GND, U1.GND1, U1.GND2; no longer JP3.1, JP3.2, JP4.P$4, JP7.1, JP7.2, U$1.GND, U$1.GND1, U$1.GND2
- net MISO: now also JP2.P$6, U1.12
- net MOSI: now also JP2.P$5, U1.11
- net SCK: now also JP3.P$5, U1.13
- net TEENSY_3V3: no longer C11.2, C13.2, C9.1, D5.3, R1.2, R2.2, SJ2.3, SJ3.3, U2.P$11, U2.P$12, U5.8, U7.3, U7.7, U7.8
- net VBAT: now also U1.VBAT; no longer U$1.VBAT
- net VBATT: now also JP5.P$3; no longer JP4.P$3
- net VUSB: now also U1.VUSB; no longer U$1.VUSB
Routing:
- net TEENSY_3V3: track 110.6 -> 0.00 mm, vias 7 -> 0
- net 5V: track 93.7 -> 0.00 mm, vias 1 -> 0
- net VBATT: track 57.7 -> 0.00 mm, vias 1 -> 0
- net RX1: track 52.8 -> 0.00 mm, vias 2 -> 0
- net TX1: track 50.0 -> 0.00 mm, vias 1 -> 0
- net GND: track 44.3 -> 0.00 mm, vias 28 -> 0
- net CMD: track 32.7 -> 0.00 mm, vias 1 -> 0
- net N$14: track 25.0 -> 0.00 mm, vias 1 -> 0
- net AUXDA: track 23.8 -> 0.00 mm, vias 1 -> 0
- net SCK: track 18.3 -> 0.00 mm, vias 2 -> 0
- net YEL_LED: track 17.5 -> 0.00 mm, vias 1 -> 0
- net BT_CMD: track 16.5 -> 0.00 mm, vias 1 -> 0
- net POW_I/O1: track 16.5 -> 0.00 mm, vias 1 -> 0
- net POW_I/O2: track 16.5 -> 0.00 mm, vias 1 -> 0
- net AUXCL: track 15.9 -> 0.00 mm, vias 1 -> 0
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- removed copper zone on layer 1, net GND
- removed copper zone on layer 16, net GND
- removed copper zone on layer 1, net N$20
- removed copper zone on layer 16, net N$25
- removed copper zone on layer 16, net N$26
- removed copper zone on layer 16, net N$28
- removed copper zone on layer 16, net N$4
Other:
- board size 38.1 x 50.8 mm -> 41.9 x 52.1 mm
- board text removed: "+"
- board text removed: "-"
- board text removed: "0"
- board text removed: "1"
- board text removed: "10"
- board text removed: "11"
- board text removed: "12"
- board text removed: "13"
- board text removed: "14"
- board text removed: "15"
- board text removed: "16"
- board text removed: "17"
- board text removed: "18"
- board text removed: "19"
- board text removed: "2"
- board text removed: "20"
- board text removed: "21"
- board text removed: "22"
- board text removed: "23"
- board text removed: "3"
- board text removed: "3v3"
- board text removed: "4"
- board text removed: "5"
- board text removed: "5V"
- board text removed: "5v"
- board text removed: "6"
- board text removed: "7"
- board text removed: "8"
- board text removed: "9"
- board text removed: "ASCL"
- board text removed: "ASDA"
- board text removed: "Aug 2013"
- board text removed: "BT"
- board text removed: "CMD"
- board text removed: "Duo/Quad"
- board text removed: "GND"
- board text removed: "IMU"
- board text removed: "INT"
- board text removed: "PWR"
- board text removed: "RX"
- board text removed: "S"
- board text removed: "Sense"
- board text removed: "TX"
- board text removed: "V0.2.4"
- board text removed: "VIN"
- board text removed: "Vin"
- board text removed: "Voltage"
- board text removed: "X"
- board text removed: "Y"
- board text removed: "Z"
- board text removed: "~"

Commit message: More work on the Tilty Omni
Parts:
- moved C13 100.6 mm to (10.2, 15.2), turned to 180 degrees
- moved D3 85.1 mm to (5.33, 6.10), turned to 180 degrees
- moved D4 80.8 mm to (23.4, 49.3)
- moved D5 78.7 mm to (17.3, 49.3)
- moved U7 74.4 mm to (8.89, 20.1)
- moved D2 70.4 mm to (5.33, 3.81), turned to 180 degrees
- moved D1 68.7 mm to (5.33, 8.38), turned to 180 degrees
- moved U4 18.6 mm to (29.5, 12.7), turned to 90 degrees
- moved R2 15.9 mm to (26.2, 30.5), turned to 180 degrees
- moved R1 11.0 mm to (26.2, 33.0), turned to 180 degrees
- moved U5 0.18 mm to (21.1, 42.3), turned to 270 degrees
Connections:
- removed net SCL: R1.1, U5.23
- removed net SDA: R2.1, U5.24
- removed net TEENSY_3V3: C2.2, U5.13
- net +3V3: now also C2.2, U5.13
- net 3V_SCL: now also R1.1, U5.23
- net 3V_SDA: now also R2.1, U5.24

Commit message: Tilty Omni updates, updated things to do
Parts:
- C5: value 0.1uF -> 4.7uF
- moved C9 106.6 mm to (31.5, 17.0)
- moved C5 105.8 mm to (34.0, 13.0)
- moved C4 105.7 mm to (37.1, 8.89)
- moved R7 97.5 mm to (14.0, 4.57), turned to 270 degrees
- moved R3 91.3 mm to (4.06, 8.38), turned to 270 degrees
- moved R4 76.4 mm to (4.06, 2.29), turned to 90 degrees
- moved R8 74.5 mm to (4.06, 5.33), turned to 270 degrees
- moved D1 2.70 mm to (7.11, 6.35)
- moved D2 2.70 mm to (7.11, 1.78)
- moved D3 2.70 mm to (7.11, 4.06)
Connections:
- removed net 5V: D2.1
- removed net N$10: U1.5
- removed net VBATT: C4.1, JP5.P$3, SJ4.1, U4.P$2
- new net 24: U1.24
- new net 25: U1.25
- new net 26: U1.26
- new net 27: U1.27
- new net 28: U1.28
- new net 29: U1.29
- new net 30: U1.30
- new net 31: U1.31
- new net 32: U1.32
- new net 33: U1.33
- new net A10: U1.A10
- new net A11: U1.A11
- new net A12: U1.A12
- new net A13: U1.A13
- net +5V: now also D2.1
- net IMU_INT: now also U1.5
- net VCC: now also C4.1, JP5.P$3, SJ4.1, U4.P$2
Routing:
- net GND: track 0.00 -> 12.0 mm
- net N$3: track 0.00 -> 2.69 mm
- net N$24: track 0.00 -> 2.37 mm
- net N$13: track 0.00 -> 2.34 mm

Commit message: Tilty PCB work
Parts:
- U1: value TEENSY_3.0_ALLPINS -> TEENSY_3.0_ALLPINSTEENSY_3.0_ALLPINS-SMD; device Teensy3.0:TEENSY_3.0_ALLPINS -> Teensy3.0:TEENSY_3.0_ALLPINS-SMD
- moved C11 114.3 mm to (35.3, 18.8), turned to 90 degrees
- moved C3 86.9 mm to (33.5, 26.9), turned to 90 degrees
- moved C1 81.4 mm to (32.8, 19.3), turned to 180 degrees
- moved C2 81.2 mm to (35.1, 30.0), turned to 90 degrees
- moved R4 34.5 mm to (38.1, 7.87)
- moved R8 32.1 mm to (36.1, 7.87)
- moved R3 30.0 mm to (34.0, 7.87)
- moved D1 23.9 mm to (31.0, 6.35), turned to 0 degrees
- moved D2 23.9 mm to (31.0, 1.78), turned to 0 degrees
- moved D3 23.9 mm to (31.0, 4.06), turned to 0 degrees
- moved U5 22.7 mm to (32.9, 22.9), turned to 0 degrees
- moved R1 7.50 mm to (33.0, 30.0), turned to 270 degrees
- moved C4 5.61 mm to (31.5, 8.38)
- moved R2 4.85 mm to (31.0, 30.0), turned to 270 degrees
- moved D4 1.48 mm to (22.1, 48.5), turned to 270 degrees
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Routing:
- net GND: track 12.0 -> 0.00 mm
- net 3V_SDA: track 0.00 -> 6.43 mm
- net 3V_SCL: track 0.00 -> 6.33 mm
- net N$3: track 2.69 -> 0.00 mm
- net N$24: track 2.37 -> 0.00 mm
- net N$13: track 2.34 -> 0.00 mm

Commit message: LOTS of work on the Tilty Omni
Parts:
- MPU_INT: value SOLDERJUMPERNO -> SOLDERJUMPERTRACE; device SparkFun-Passives:SJ_2S-NO -> SparkFun-Passives:SJ_2S-TRACE
- moved MPU_INT 90.6 mm to (33.5, 27.4), flipped to the bottom, turned to 180 degrees
- moved R5 78.8 mm to (4.57, 60.2)
- moved R6 73.0 mm to (3.05, 55.9)
- moved SJ5 70.5 mm to (9.40, 60.7)
- moved SJ1 63.8 mm to (13.0, 59.4)
- moved SJ4 58.3 mm to (22.1, 58.9)
- moved JP9 40.6 mm to (12.2, 55.4)
- moved C9 12.7 mm to (19.1, 14.7)
- moved C2 11.7 mm to (31.0, 19.1)
- moved C11 11.2 mm to (35.1, 30.0), turned to 270 degrees
- moved U2 10.3 mm to (21.0, 17.8), turned to 180 degrees
- moved R1 5.92 mm to (35.3, 35.4), turned to 0 degrees
- moved R2 5.21 mm to (35.3, 32.9), turned to 0 degrees
- moved C3 3.11 mm to (32.9, 30.0)
- moved C1 2.05 mm to (34.8, 19.1), turned to 270 degrees
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Connections:
- removed net 33: U1.33
- removed net A13: U1.A13
- removed net AUX_SCL: JP3.P$7
- removed net AUX_SDA: JP3.P$6
- removed net MPU_INT: MPU_INT.1
- new net 14/A0: JP3.P$4, U1.14/A0
- new net 15/A1: JP3.P$3, U1.15/A1
- new net 5/PWM: JP1.P$7, JP6.14, U1.5
- new net 6/PWM: JP6.13, U1.6
- new net N$30: JP7.1
- new net N$31: JP7.2
- new net N$32: JP7.3
- new net N$33: JP7.4
- new net N$34: JP7.5
- new net N$35: JP7.6
- new net N$36: JP7.7
- new net N$37: JP7.8
- new net N$38: JP7.9
- new net N$39: JP7.10
- new net N$40: JP7.11
- new net N$41: JP7.12
- new net N$42: JP7.13
- new net N$43: JP7.14
- new net N$44: JP7.15
- new net N$45: JP7.16
- new net N$46: JP7.17
- new net N$47: JP7.18
- new net N$48: JP7.19
- new net N$49: JP7.20
- net 10/TX2: now also JP6.9
- net 24: now also JP6.5
- net 25: now also JP6.4
- net 26: now also JP6.3
- net 27: now also JP6.2
- net 28: now also JP6.1; no longer U1.28
- net 4/PWM: now also JP6.15
- net 7/RX3: now also JP6.12
- net 8/TX3: now also JP6.11
- net 9/RX2: now also JP6.10
- net AUXCL: now also JP3.P$7
- net AUXDA: now also JP3.P$6
- net BATT_SENSE: now also U1.A13; no longer JP3.P$4, U1.14/A0
- net BLUETOOTH_RX: now also JP6.19
- net BLUETOOTH_TX: now also JP6.18
- net BT_CMD: now also U1.28; no longer JP3.P$3, U1.15/A1
- net GND: now also JP6.20
- net IMU_INT: now also MPU_INT.1, U1.33; no longer JP1.P$7, U1.5
- net MEMORY_CS: no longer U1.6
- net MISO: now also JP6.7
- net MOSI: now also JP6.8
- net SCK: now also JP6.6
- net SERVO_1: now also JP6.17
- net SERVO_2: now also JP6.16
Routing:
- net +3V3: track 0.00 -> 39.1 mm, vias 0 -> 4
- net GND: track 0.00 -> 28.8 mm
- net AUXCL: track 0.00 -> 13.7 mm, vias 0 -> 1
- net AUXDA: track 0.00 -> 13.1 mm, vias 0 -> 1
- net 14/A0: track 0.00 -> 11.0 mm, vias 0 -> 1
- net 15/A1: track 0.00 -> 10.4 mm, vias 0 -> 1
- net SCK: track 0.00 -> 10.1 mm
- net 5V_SCL: track 0.00 -> 10.1 mm, vias 0 -> 1
- net 3V_SCL: track 6.33 -> 15.9 mm
- net 5V_SDA: track 0.00 -> 9.24 mm, vias 0 -> 1
- net 3V_SDA: track 6.43 -> 13.3 mm, vias 0 -> 1
- net N$2: track 0.00 -> 3.65 mm
- net N$1: track 0.00 -> 3.51 mm

Commit message: Lots more Tilty Omni work!
Parts:
- moved JP9 58.0 mm to (44.5, 7.11), turned to 270 degrees
- moved SJ5 57.2 mm to (29.7, 7.24), flipped to the bottom
- moved R5 47.6 mm to (20.1, 15.2)
- moved R6 46.1 mm to (22.6, 14.2), turned to 90 degrees
- moved SJ4 46.0 mm to (19.7, 13.0), turned to 90 degrees
- moved SJ1 16.4 mm to (21.1, 45.2)
- moved D4 13.9 mm to (35.6, 45.0)
- moved R7 13.6 mm to (27.4, 7.87)
- moved C9 13.4 mm to (10.9, 25.4), turned to 90 degrees
- moved D5 11.9 mm to (6.60, 45.2), turned to 0 degrees
- moved U7 7.38 mm to (9.65, 13.0), turned to 90 degrees
- moved C13 4.35 mm to (14.5, 14.2), turned to 270 degrees
Connections:
- removed net 28: JP6.1
- removed net N$30: JP7.1
- removed net N$31: JP7.2
- removed net N$32: JP7.3
- removed net N$33: JP7.4
- removed net N$34: JP7.5
- removed net N$35: JP7.6
- removed net N$36: JP7.7
- removed net N$37: JP7.8
- removed net N$38: JP7.9
- removed net N$39: JP7.10
- removed net N$40: JP7.11
- removed net N$41: JP7.12
- removed net N$42: JP7.13
- removed net N$43: JP7.14
- removed net N$44: JP7.15
- removed net N$45: JP7.16
- removed net N$46: JP7.17
- removed net N$47: JP7.18
- removed net N$48: JP7.19
- removed net N$49: JP7.20
- net +3V3: now also JP7.18
- net +5V: now also JP7.20
- net 14/A0: now also JP7.8
- net 15/A1: now also JP7.9
- net 20/A6: now also JP7.14
- net 21/A7: now also JP7.15
- net 27: no longer U1.27
- net 29: now also JP7.1
- net 30: now also JP7.2
- net 31: now also JP7.3
- net 32: now also JP7.4
- net 3V_SCL: now also JP7.13
- net 3V_SDA: now also JP7.12
- net 5V_SCL: now also JP7.10, JP7.11
- net 6/PWM: now also JP1.P$8
- net A10: now also JP7.7
- net A11: now also JP7.6
- net A12: now also JP7.5
- net AGND: now also JP7.19
- net BLUETOOTH_RX: now also U2.P$1
- net BLUETOOTH_TX: now also U2.P$2
- net MEMORY_CS: now also JP6.1, U1.27; no longer JP1.P$8
- net RX1: no longer U2.P$1
- net SERVO_3: now also JP7.16
- net SERVO_4: now also JP7.17
- net TX1: no longer U2.P$2
Routing:
- net BLUETOOTH_RX: track 0.00 -> 48.7 mm
- net BLUETOOTH_TX: track 0.00 -> 44.7 mm, vias 0 -> 1
- net +3V3: track 39.1 -> 71.4 mm, vias 4 -> 7
- net SCK: track 10.1 -> 41.4 mm
- net GND: track 28.8 -> 55.4 mm, vias 0 -> 3
- net BATT_SENSE: track 0.00 -> 24.9 mm, vias 0 -> 2
- net VCC: track 0.00 -> 23.3 mm
- net MISO: track 0.00 -> 20.0 mm, vias 0 -> 2
- net MEMORY_CS: track 0.00 -> 19.0 mm, vias 0 -> 2
- net MOSI: track 0.00 -> 17.5 mm
- net 10/TX2: track 0.00 -> 13.2 mm
- net 9/RX2: track 0.00 -> 13.1 mm
- net IMU_INT: track 0.00 -> 11.7 mm, vias 0 -> 1
- net N$16: track 0.00 -> 11.5 mm
- net SERVO_2: track 0.00 -> 3.99 mm
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
Commit message: GPS breakout work, and minor Tilty Omni changes
Parts:
- moved SJ1 14.5 mm to (6.60, 45.2), flipped to the bottom
- moved D5 12.9 mm to (15.7, 54.4)
- moved JP7 0.13 mm to (40.6, 1.91)
Routing:
- net BLUETOOTH_RX: track 48.7 -> 59.4 mm
- net +5V: track 0.00 -> 8.53 mm
- net SERVO_1: track 3.74 -> 12.3 mm
- net 6/PWM: track 3.86 -> 12.3 mm
- net 4/PWM: track 3.86 -> 12.3 mm
- net BLUETOOTH_TX: track 44.7 -> 53.0 mm
- net 5/PWM: track 3.99 -> 12.3 mm
- net SERVO_2: track 3.99 -> 12.3 mm

Commit message: Tilty Omni work
Connections:
- removed net 27: JP6.2
- net BT_CMD: now also JP6.1
- net MEMORY_CS: now also JP6.2; no longer JP6.1
Routing:
- net 7/RX3: track 0.00 -> 12.9 mm
- net 8/TX3: track 0.00 -> 12.9 mm
- net MOSI: track 17.5 -> 18.4 mm
- net MISO: track 20.0 -> 20.6 mm
Changed lines of the file:
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@@
 <contactref element="SJ5" pad="1"/>
 <contactref element="U1" pad="28"/>
+<contactref element="JP6" pad="1"/>
 <wire x1="30.1299" y1="7.239" x2="19.685" y2="20.32" width="0" layer="19" extent="1-16"/>
+<wire x1="1.3335" y1="1.905" x2="19.685" y2="20.32" width="0" layer="19" extent="1-1"/>
 </signal>
 <signal name="N$3">
@@
 <contactref element="U1" pad="12"/>
 <contactref element="JP6" pad="7"/>
-<via x="10.16" y="17.78" extent="1-16" drill="0.3302"/>
-<wire x1="4.445" y1="16.383" x2="9.779" y2="16.383" width="0.2032" layer="16"/>
-<wire x1="9.779" y1="16.383" x2="10.16" y2="16.764" width="0.2032" layer="16"/>
-<wire x1="10.16" y1="16.764" x2="10.16" y2="17.78" width="0.2032" layer="16"/>
-<wire x1="10.16" y1="17.78" x2="13.335" y2="17.78" width="0.2032" layer="1"/>
+<via x="10.033" y="17.78" extent="1-16" drill="0.3302"/>
+<wire x1="10.033" y1="17.78" x2="13.335" y2="17.78" width="0.2032" layer="1"/>
 <wire x1="1.3335" y1="17.145" x2="3.683" y2="17.145" width="0.2032" layer="1"/>
 <wire x1="3.683" y1="17.145" x2="4.445" y2="16.383" width="0.2032" layer="1"/>
-<via x="9.779" y="12.319" extent="1-16" drill="0.3302"/>
-<wire x1="9.779" y1="12.319" x2="12.2682" y2="12.319" width="0.2032" layer="1"/>
-<wire x1="9.779" y1="12.319" x2="9.779" y2="16.383" width="0.2032" layer="16"/>
+<via x="10.033" y="12.319" extent="1-16" drill="0.3302"/>
+<wire x1="10.033" y1="12.319" x2="12.2682" y2="12.319" width="0.2032" layer="1"/>
+<wire x1="10.033" y1="17.78" x2="5.842" y2="17.78" width="0.2032" layer="16"/>
+<wire x1="5.842" y1="17.78" x2="4.445" y2="16.383" width="0.2032" layer="16"/>
+<wire x1="10.033" y1="12.319" x2="10.033" y2="17.78" width="0.2032" layer="16"/>
 </signal>
 <signal name="SCK">
@@
 <contactref element="U1" pad="11"/>
 <contactref element="JP6" pad="8"/>
-<wire x1="7.0358" y1="14.859" x2="7.0358" y2="18.4912" width="0.2032" layer="1"/>
-<wire x1="7.0358" y1="18.4912" x2="6.604" y2="18.923" width="0.2032" layer="1"/>
-<wire x1="6.604" y1="18.923" x2="4.318" y2="18.923" width="0.2032" layer="1"/>
-<wire x1="7.0358" y1="18.4912" x2="7.0612" y2="18.4912" width="0.2032" layer="1"/>
-<wire x1="7.0612" y1="18.4912" x2="7.493" y2="18.923" width="0.2032" layer="1"/>
-<wire x1="7.493" y1="18.923" x2="7.493" y2="19.939" width="0.2032" layer="1"/>
-<wire x1="7.493" y1="19.939" x2="7.874" y2="20.32" width="0.2032" layer="1"/>
-<wire x1="7.874" y1="20.32" x2="13.335" y2="20.32" width="0.2032" layer="1"/>
+<wire x1="6.0198" y1="18.4912" x2="5.588" y2="18.923" width="0.2032" layer="1"/>
+<wire x1="5.588" y1="18.923" x2="4.318" y2="18.923" width="0.2032" layer="1"/>
+<wire x1="6.0198" y1="18.4912" x2="6.0452" y2="18.4912" width="0.2032" layer="1"/>
+<wire x1="6.0452" y1="18.4912" x2="6.477" y2="18.923" width="0.2032" layer="1"/>
+<wire x1="6.477" y1="18.923" x2="6.477" y2="19.939" width="0.2032" layer="1"/>
+<wire x1="6.477" y1="19.939" x2="6.858" y2="20.32" width="0.2032" layer="1"/>
+<wire x1="6.858" y1="20.32" x2="13.335" y2="20.32" width="0.2032" layer="1"/>
 <wire x1="1.3335" y1="19.685" x2="3.556" y2="19.685" width="0.2032" layer="1"/>
 <wire x1="3.556" y1="19.685" x2="4.318" y2="18.923" width="0.2032" layer="1"/>
+<wire x1="6.0198" y1="18.4912" x2="6.0198" y2="15.0622" width="0.2032" layer="1"/>
+<wire x1="6.0198" y1="15.0622" x2="6.096" y2="14.986" width="0.2032" layer="1"/>
+<wire x1="6.096" y1="14.986" x2="6.9088" y2="14.986" width="0.2032" layer="1"/>
+<wire x1="6.9088" y1="14.986" x2="7.0358" y2="14.859" width="0.2032" layer="1"/>
 </signal>
 <signal name="N$13">
@@
 <contactref element="U1" pad="8"/>
 <contactref element="JP6" pad="11"/>
-<wire x1="4.572" y1="26.543" x2="13.335" y2="27.94" width="0" layer="19" extent="1-1"/>
-<wire x1="1.3335" y1="27.305" x2="4.572" y2="26.543" width="0" layer="19" extent="1-1"/>
+<wire x1="13.335" y1="27.94" x2="5.969" y2="27.94" width="0.254" layer="1"/>
+<wire x1="5.969" y1="27.94" x2="4.572" y2="26.543" width="0.254" layer="1"/>
+<wire x1="4.572" y1="26.543" x2="3.81" y2="27.305" width="0.2032" layer="1"/>
+<wire x1="3.81" y1="27.305" x2="1.3335" y2="27.305" width="0.2032" layer="1"/>
 </signal>
 <signal name="7/RX3">
@@
 <contactref element="U1" pad="7"/>
 <contactref element="JP6" pad="12"/>
-<wire x1="4.318" y1="29.083" x2="13.335" y2="30.48" width="0" layer="19" extent="1-1"/>
-<wire x1="1.3335" y1="29.845" x2="4.318" y2="29.083" width="0" layer="19" extent="1-1"/>
+<wire x1="13.335" y1="30.48" x2="5.715" y2="30.48" width="0.254" layer="1"/>
+<wire x1="5.715" y1="30.48" x2="4.318" y2="29.083" width="0.254" layer="1"/>
+<wire x1="4.318" y1="29.083" x2="3.556" y2="29.845" width="0.2032" layer="1"/>
+<wire x1="3.556" y1="29.845" x2="1.3335" y2="29.845" width="0.2032" layer="1"/>
 </signal>
 <signal name="MEMORY_CS">
 <contactref element="U7" pad="1"/>
 <contactref element="U1" pad="27"/>
-<contactref element="JP6" pad="1"/>
 <via x="19.685" y="22.86" extent="1-16" drill="0.3302"/>
 <wire x1="19.685" y1="22.86" x2="17.526" y2="22.86" width="0.2032" layer="16"/>
@@
 <wire x1="17.145" y1="22.479" x2="17.145" y2="11.049" width="0.2032" layer="16"/>
 <wire x1="12.2682" y1="11.049" x2="17.145" y2="11.049" width="0.2032" layer="1"/>
-<wire x1="1.3335" y1="1.905" x2="12.2682" y2="11.049" width="0" layer="19" extent="1-1"/>
+<contactref element="JP6" pad="2"/>
+<wire x1="1.3335" y1="4.445" x2="12.2682" y2="11.049" width="0" layer="19" extent="1-1"/>
 </signal>
 <signal name="IMU_INT">
@@
 <contactref element="D2" pad="1"/>
 <contactref element="JP7" pad="20"/>
+<wire x1="32.258" y1="50.673" x2="38.608" y2="50.673" width="0.2032" layer="1"/>
+<wire x1="38.608" y1="50.673" x2="39.116" y2="50.165" width="0.2032" layer="1"/>
+<wire x1="39.116" y1="50.165" x2="40.5765" y2="50.165" width="0.2032" layer="1"/>
 <wire x1="34.61" y1="43.958" x2="32.258" y2="50.673" width="0" layer="19" extent="1-1"/>
 <wire x1="33.8582" y1="14.986" x2="34.61" y2="43.958" width="0" layer="19" extent="1-1"/>
@@
 <wire x1="30.138" y1="1.778" x2="33.694" y2="12.7" width="0" layer="19" extent="1-1"/>
 <wire x1="44.323" y1="3.302" x2="33.694" y2="12.7" width="0" layer="19" extent="1-1"/>
-<wire x1="32.258" y1="50.673" x2="38.608" y2="50.673" width="0.2032" layer="1"/>
-<wire x1="38.608" y1="50.673" x2="39.116" y2="50.165" width="0.2032" layer="1"/>
-<wire x1="39.116" y1="50.165" x2="40.5765" y2="50.165" width="0.2032" layer="1"/>
 </signal>
 <signal name="VCC">
@@
 <wire x1="1.3335" y1="6.985" x2="19.685" y2="25.4" width="0" layer="19" extent="1-1"/>
 </signal>
-<signal name="27">
-<contactref element="JP6" pad="2"/>
-</signal>
 <signal name="29">
