File: Tilty Hardware/Board Files/GPS Adapter/Eagle PCB Files/GPS breakout.brd (EAGLE design)
At the start: 38.1 x 50.8 mm, 10 parts, among them U1 XBEE-1XBEE-1_LOCK, U2 LM2931, U3 V_REG_LDOSMD

Commit message: Nearly finished RC Receiver add-on prototype, worked on TiltyIMU library
Parts:
- removed U3: V_REG_LDOSMD, SparkFun-PowerIC:SOT23-5
- flipped C2 to the top
- flipped C3 to the top
- flipped U2 to the top
Connections:
- net 3V3: no longer C1.1, U3.5
- net 5V: no longer U3.1, U3.3
- net GND: no longer C1.2, U3.2
Changed lines of the file:
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@@
 </autorouter>
 <elements>
-<element name="U2" library="on-semiconductor" package="TO263" value="LM2931" x="19.05" y="44.5135" smashed="yes" rot="MR0">
-<attribute name="COST" value="0.53" x="19.05" y="44.5135" size="1.778" layer="28" rot="MR0" display="off"/>
+<element name="U2" library="on-semiconductor" package="TO263" value="LM2931" x="19.05" y="44.5135" smashed="yes">
+<attribute name="COST" value="0.53" x="19.05" y="44.5135" size="1.778" layer="27" display="off"/>
 </element>
-<element name="C2" library="resistor" package="C0603" value="0.1uF" x="22.987" y="40.259" smashed="yes" rot="MR90"/>
-<element name="C3" library="resistor" package="C0603" value="0.1uF" x="15.113" y="40.259" smashed="yes" rot="MR90"/>
+<element name="C2" library="resistor" package="C0603" value="0.1uF" x="22.987" y="40.259" smashed="yes" rot="R90"/>
+<element name="C3" library="resistor" package="C0603" value="0.1uF" x="15.113" y="40.259" smashed="yes" rot="R90"/>
 <element name="JP1" library="pinhead" package="1X08_NO_SS_LOCKING" value="" x="7.62" y="40.513" smashed="yes" rot="R90">
 <attribute name="VALUE" x="10.795" y="30.353" size="1.27" layer="27" rot="R90"/>
@@
 <attribute name="VALUE" x="10.16" y="7.62" size="0.4064" layer="27"/>
 </element>
-<element name="U3" library="SparkFun-PowerIC" package="SOT23-5" value="V_REG_LDOSMD" x="-2.54" y="2.54">
-<attribute name="PART#" value="TLV71333PDBVR" x="-2.54" y="2.54" size="1.778" layer="27" display="off"/>
-</element>
 <element name="C1" library="resistor" package="C0603" value="0.1uF" x="-2.54" y="-2.54"/>
 </elements>
@@
 <contactref element="JP6" pad="1"/>
 <contactref element="U1" pad="10"/>
-<contactref element="U3" pad="2"/>
-<contactref element="C1" pad="2"/>
-<wire x1="22.987" y1="41.109" x2="30.353" y2="46.863" width="0" layer="19" extent="16-16"/>
-<wire x1="19.05" y1="47.3075" x2="22.987" y2="41.109" width="0" layer="19" extent="16-16"/>
-<wire x1="15.113" y1="41.109" x2="19.05" y2="47.3075" width="0" layer="19" extent="16-16"/>
-<wire x1="35.433" y1="11.303" x2="22.987" y2="41.109" width="0" layer="19" extent="16-16"/>
+<wire x1="22.987" y1="41.109" x2="30.353" y2="46.863" width="0" layer="19" extent="1-1"/>
+<wire x1="19.05" y1="47.3075" x2="22.987" y2="41.109" width="0" layer="19" extent="1-1"/>
+<wire x1="15.113" y1="41.109" x2="19.05" y2="47.3075" width="0" layer="19" extent="1-1"/>
+<wire x1="35.433" y1="11.303" x2="22.987" y2="41.109" width="0" layer="19" extent="1-1"/>
 <wire x1="8.2278" y1="8.35" x2="35.433" y2="11.303" width="0" layer="19" extent="1-1"/>
 <wire x1="2.413" y1="11.303" x2="8.2278" y2="8.35" width="0" layer="19" extent="1-1"/>
-<wire x1="-2.54" y1="1.2399" x2="2.413" y2="11.303" width="0" layer="19" extent="1-1"/>
-<wire x1="-1.69" y1="-2.54" x2="-2.54" y2="1.2399" width="0" layer="19" extent="1-1"/>
 </signal>
 <signal name="SCL" class="4">
@@
 <contactref element="C2" pad="1"/>
 <contactref element="JP2" pad="2"/>
-<wire x1="21.336" y1="40.1193" x2="22.987" y2="39.409" width="0" layer="19" extent="16-16"/>
-<wire x1="2.667" y1="13.843" x2="21.336" y2="40.1193" width="0" layer="19" extent="16-16"/>
+<wire x1="16.764" y1="40.1193" x2="22.987" y2="39.409" width="0" layer="19" extent="16-16"/>
+<wire x1="2.667" y1="13.843" x2="16.764" y2="40.1193" width="0" layer="19" extent="16-16"/>
 </signal>
 <signal name="5V">
@@
 <contactref element="C3" pad="1"/>
 <contactref element="JP5" pad="8"/>
-<contactref element="U3" pad="1"/>
-<contactref element="U3" pad="3"/>
-<wire x1="16.764" y1="40.1193" x2="30.607" y2="49.403" width="0" layer="19" extent="16-16"/>
-<wire x1="15.113" y1="39.409" x2="16.764" y2="40.1193" width="0" layer="19" extent="16-16"/>
-<wire x1="-1.59" y1="1.2399" x2="15.113" y2="39.409" width="0" layer="19" extent="1-16"/>
-<wire x1="-3.49" y1="1.2399" x2="-1.59" y2="1.2399" width="0" layer="19" extent="1-1"/>
+<wire x1="21.336" y1="40.1193" x2="30.607" y2="49.403" width="0" layer="19" extent="1-1"/>
+<wire x1="15.113" y1="39.409" x2="21.336" y2="40.1193" width="0" layer="19" extent="1-1"/>
 </signal>
 <signal name="N$23">
@@
 </signal>
 <signal name="3V3" class="3">
-<contactref element="U3" pad="5"/>
 <contactref element="JP1" pad="8"/>
-<contactref element="C1" pad="1"/>
-<wire x1="-3.49" y1="3.8401" x2="7.747" y2="49.403" width="0" layer="19" extent="1-1"/>
-<wire x1="-3.39" y1="-2.54" x2="-3.49" y2="3.8401" width="0" layer="19" extent="1-1"/>
 </signal>
 </signals>

Commit message: GPS breakout work, and minor Tilty Omni changes
Connections:
- removed net N$10: JP6.8
- removed net N$23: JP6.7
- net 5V: no longer JP5.8
Changed lines of the file:
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@@
 <contactref element="C3" pad="2"/>
 <contactref element="C2" pad="2"/>
-<contactref element="JP5" pad="7"/>
 <contactref element="JP2" pad="1"/>
 <contactref element="JP6" pad="1"/>
 <contactref element="U1" pad="10"/>
+<contactref element="JP5" pad="7"/>
 <wire x1="22.987" y1="41.109" x2="30.353" y2="46.863" width="0" layer="19" extent="1-1"/>
 <wire x1="19.05" y1="47.3075" x2="22.987" y2="41.109" width="0" layer="19" extent="1-1"/>
@@
 <contactref element="U2" pad="P$3"/>
 <contactref element="C3" pad="1"/>
-<contactref element="JP5" pad="8"/>
-<wire x1="21.336" y1="40.1193" x2="30.607" y2="49.403" width="0" layer="19" extent="1-1"/>
 <wire x1="15.113" y1="39.409" x2="21.336" y2="40.1193" width="0" layer="19" extent="1-1"/>
 </signal>
-<signal name="N$23">
-<contactref element="JP6" pad="7"/>
-</signal>
-<signal name="N$10">
-<contactref element="JP6" pad="8"/>
-</signal>
 <signal name="VDD">
