File: Tilty Hardware/Board Files/Tilty Duo and Quad/V0.2.5/Eagle PCB Files/TiltyDuo.brd (EAGLE design)
At the start: 38.1 x 50.8 mm, 50 parts, among them U1 TEENSY_3.0_OUTER-PINS28-DIP_S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, U2 HC-09_BREAKOUT, U3 MPL3115A2LGA8, U4 LM2931, U5 MPU-6050, U6 HMC5883LSMD, U7 SPI_FLASH-X25XXSMD

Commit message: Minor changes
Added current limit resistor to zener shunt on Tilty Duo/Quad.
Added power supply solder jumper to Advanced IMU altimeter.
Parts:
- added R9: (no value), resistor:R0603
Connections:
- new net N$22: D5.1, R9.2
- net GND: now also R9.1; no longer D5.1
Routing:
- net N$22: track 0.00 -> 1.20 mm
Changed lines of the file:
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@@
 <attribute name="VALUE" x="16.256" y="18.9865" size="0.4064" layer="27"/>
+</element>
+<element name="R9" library="resistor" package="R0603" value="" x="14.9225" y="45.72" smashed="yes" rot="MR90">
+<attribute name="VALUE" x="12.8905" y="44.831" size="1.27" layer="28" rot="MR90"/>
 </element>
 </elements>
@@
 <via x="10.541" y="15.494" extent="1-16" drill="0.3302"/>
 <via x="36.449" y="27.7495" extent="1-16" drill="0.3302"/>
-<contactref element="D5" pad="1"/>
 <contactref element="JP4" pad="P$2"/>
 <contactref element="JP3" pad="P$8"/>
@@
 <wire x1="33.997" y1="12.7" x2="33.655" y2="13.042" width="0.27431875" layer="16"/>
 <contactref element="C6" pad="2"/>
+<contactref element="R9" pad="1"/>
 </signal>
 <signal name="SCL" class="4">
@@
 <wire x1="17.907" y1="20.828" x2="18.542" y2="20.828" width="0.2032" layer="1"/>
 </signal>
+<signal name="N$22">
+<contactref element="D5" pad="1"/>
+<contactref element="R9" pad="2"/>
+<wire x1="14.92" y1="47.768" x2="14.92" y2="46.5725" width="0.381" layer="16"/>
+<wire x1="14.92" y1="46.5725" x2="14.9225" y2="46.57" width="0.381" layer="16"/>
+</signal>
 </signals>

Commit message: Lots of little updates!
Parts:
- removed D4: (no value), SparkFun-DiscreteSemi:SOT23-3
Connections:
- removed net N$15: D4.3, U1.P$15
- net 5V: now also U1.P$15; no longer D4.1
Routing:
- net N$15: track 2.61 -> 0.00 mm
- net 5V: track 99.7 -> 100.7 mm
Changed lines of the file:
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@@
 <attribute name="VALUE" x="19.939" y="12.7635" size="0.4064" layer="27" rot="R90"/>
-</element>
-<element name="D4" library="SparkFun-DiscreteSemi" package="SOT23-3" value="" x="24.13" y="48.768" smashed="yes" rot="MR0">
-<attribute name="VALUE" x="25.146" y="48.5775" size="0.4064" layer="28" rot="MR0"/>
-<attribute name="PART#" value="BAT54FSTR-ND" x="24.13" y="48.768" size="1.778" layer="28" rot="MR0" display="off"/>
 </element>
 <element name="D5" library="SparkFun-DiscreteSemi" package="SOT23-3" value="" x="13.97" y="48.768" smashed="yes" rot="MR0">
@@
 <wire x1="17.145" y1="42.545" x2="16.764" y2="42.164" width="0.381" layer="16"/>
 <wire x1="16.764" y1="42.164" x2="16.764" y2="40.1193" width="0.381" layer="16"/>
-<contactref element="D4" pad="1"/>
 <wire x1="23.368" y1="43.18" x2="23.368" y2="44.704" width="0.381" layer="16"/>
 <wire x1="23.368" y1="44.704" x2="23.876" y2="45.212" width="0.381" layer="16"/>
 <wire x1="23.876" y1="45.212" x2="24.511" y2="45.212" width="0.381" layer="16"/>
 <wire x1="24.511" y1="45.212" x2="25.019" y2="45.72" width="0.381" layer="16"/>
-<wire x1="25.019" y1="45.72" x2="25.019" y2="47.707" width="0.381" layer="16"/>
-<wire x1="25.019" y1="47.707" x2="25.08" y2="47.768" width="0.381" layer="16"/>
-<wire x1="25.08" y1="47.768" x2="25.67" y2="47.768" width="0.381" layer="16"/>
-<wire x1="25.67" y1="47.768" x2="26.162" y2="48.26" width="0.381" layer="16"/>
 <contactref element="JP4" pad="P$1"/>
 <wire x1="30.353" y1="49.403" x2="29.21" y2="48.26" width="0.381" layer="16"/>
@@
 <wire x1="16.51" y1="36.0807" x2="21.5138" y2="36.0807" width="0.381" layer="16"/>
 <wire x1="21.5138" y1="36.0807" x2="21.59" y2="36.0045" width="0.381" layer="16"/>
+<contactref element="U1" pad="P$15"/>
+<wire x1="25.019" y1="45.72" x2="25.019" y2="47.117" width="0.381" layer="16"/>
+<wire x1="25.019" y1="47.117" x2="26.035" y2="48.133" width="0.381" layer="16"/>
+<wire x1="26.035" y1="48.133" x2="26.162" y2="48.26" width="0.381" layer="16"/>
+<wire x1="26.543" y1="49.403" x2="26.543" y2="48.641" width="0.381" layer="16"/>
+<wire x1="26.543" y1="48.641" x2="26.162" y2="48.26" width="0.381" layer="16"/>
 </signal>
 <signal name="N$7">
@@
 <wire x1="2.667" y1="21.463" x2="11.43" y2="21.463" width="0.254" layer="1"/>
 </signal>
-<signal name="N$15">
-<contactref element="D4" pad="3"/>
-<contactref element="U1" pad="P$15"/>
-<wire x1="24.13" y1="49.868" x2="26.078" y2="49.868" width="0.381" layer="16"/>
-<wire x1="26.078" y1="49.868" x2="26.543" y2="49.403" width="0.381" layer="16"/>
-</signal>
 <signal name="N$17" class="3">

Commit message: Minor changes to Duo/Quad silkscreen
Parts:
- moved R9 1.02 mm to (13.9, 45.7)
Routing:
- net N$22: track 1.20 -> 2.01 mm
Other:
- board text removed: "Duo/Quad"
- board text removed: "Sep 2013"
- board text removed: "V0.2.5"
Changed lines of the file:
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@@
 <layer number="19" name="Unrouted" color="6" fill="1" visible="yes" active="yes"/>
 <layer number="20" name="Dimension" color="15" fill="1" visible="yes" active="yes"/>
-<layer number="21" name="tPlace" color="16" fill="1" visible="yes" active="yes"/>
-<layer number="22" name="bPlace" color="14" fill="1" visible="yes" active="yes"/>
-<layer number="23" name="tOrigins" color="15" fill="1" visible="yes" active="yes"/>
-<layer number="24" name="bOrigins" color="15" fill="1" visible="yes" active="yes"/>
+<layer number="21" name="tPlace" color="10" fill="1" visible="no" active="yes"/>
+<layer number="22" name="bPlace" color="2" fill="1" visible="no" active="yes"/>
+<layer number="23" name="tOrigins" color="15" fill="1" visible="no" active="yes"/>
+<layer number="24" name="bOrigins" color="15" fill="1" visible="no" active="yes"/>
 <layer number="25" name="tNames" color="14" fill="1" visible="yes" active="yes"/>
 <layer number="26" name="bNames" color="6" fill="1" visible="yes" active="yes"/>
@@
 <layer number="49" name="Reference" color="7" fill="1" visible="no" active="yes"/>
 <layer number="50" name="dxf" color="7" fill="1" visible="no" active="no"/>
-<layer number="51" name="tDocu" color="15" fill="1" visible="yes" active="yes"/>
-<layer number="52" name="bDocu" color="7" fill="1" visible="yes" active="yes"/>
+<layer number="51" name="tDocu" color="15" fill="1" visible="no" active="yes"/>
+<layer number="52" name="bDocu" color="7" fill="1" visible="no" active="yes"/>
 <layer number="53" name="tGND_GNDA" color="7" fill="9" visible="no" active="no"/>
 <layer number="54" name="bGND_GNDA" color="1" fill="9" visible="no" active="no"/>
@@
 <text x="24.892" y="4.2545" size="1.778" layer="26" ratio="10" rot="MR0" align="center-left">TX</text>
 <text x="9.525" y="47.879" size="1.016" layer="25" ratio="12" rot="R90" align="center-left">3v3</text>
-<text x="19.12359375" y="46.051375" size="1.2065" layer="25" ratio="12" align="center">Duo/Quad</text>
-<text x="19.177" y="42.926" size="1.27" layer="25" ratio="12" align="center">V0.2.5</text>
 <text x="28.956" y="6.985" size="1.2192" layer="25" ratio="12" align="center-left">BT</text>
 <text x="4.445" y="10.16" size="1.016" layer="26" ratio="10" rot="MR75" align="center-left">GND</text>
@@
 <text x="5.715" y="34.163" size="1.778" layer="25" ratio="10" align="center-right">5</text>
 <text x="5.715" y="31.623" size="1.778" layer="25" ratio="10" align="center-right">6</text>
-<circle x="29.972" y="28.6385" radius="0.3302" width="0.2286" layer="26"/>
 <text x="19.685" y="13.843" size="1.016" layer="25" font="vector" ratio="12">Voltage</text>
 <text x="19.685" y="12.573" size="1.016" layer="25" font="vector" ratio="12">Sense</text>
@@
 <rectangle x1="12.4457375" y1="2.670165625" x2="12.46605625" y2="2.690484375" layer="25" rot="R285"/>
 <text x="5.140959375" y="2.96671875" size="1.905" layer="25" font="vector" ratio="17" rot="R320">IMU</text>
-<text x="15.367" y="38.608" size="1.016" layer="25" font="vector" ratio="12">Sep 2013</text>
 <text x="5.7785" y="41.783" size="1.27" layer="26" ratio="15" rot="MR0" align="center">S</text>
 <text x="5.7785" y="39.37" size="1.27" layer="26" ratio="15" rot="MR0" align="center">+</text>
@@
 <circle x="19.05" y="24.892" radius="0.0635" width="0.254" layer="25"/>
 <text x="19.304" y="20.066" size="1.143" layer="25" ratio="15">Mag</text>
+<wire x1="2.032" y1="45.466" x2="2.032" y2="45.5295" width="0.2032" layer="26"/>
+<wire x1="2.032" y1="45.5295" x2="2.286" y2="45.7835" width="0.2032" layer="26" curve="-90"/>
+<wire x1="2.286" y1="45.7835" x2="3.81" y2="45.7835" width="0.2032" layer="26"/>
+<wire x1="4.064" y1="45.466" x2="4.064" y2="45.5295" width="0.2032" layer="26"/>
+<wire x1="4.064" y1="45.5295" x2="3.81" y2="45.7835" width="0.2032" layer="26" curve="90"/>
+<wire x1="4.064" y1="44.069" x2="4.064" y2="44.0055" width="0.2032" layer="26"/>
+<wire x1="4.064" y1="44.0055" x2="3.81" y2="43.7515" width="0.2032" layer="26" curve="-90"/>
+<wire x1="3.81" y1="43.7515" x2="2.286" y2="43.7515" width="0.2032" layer="26"/>
+<wire x1="2.032" y1="44.069" x2="2.032" y2="44.0055" width="0.2032" layer="26"/>
+<wire x1="2.032" y1="44.0055" x2="2.286" y2="43.7515" width="0.2032" layer="26" curve="90"/>
+<circle x="29.591" y="25.2095" radius="0.0254" width="0.381" layer="26"/>
+<circle x="5.1435" y="19.939" radius="0.0254" width="0.381" layer="26"/>
+<wire x1="20.32" y1="20.193" x2="20.701" y2="19.812" width="0.254" layer="26"/>
+<wire x1="20.701" y1="23.368" x2="21.082" y2="23.749" width="0.254" layer="26"/>
+<wire x1="35.2425" y1="8.636" x2="35.4965" y2="8.89" width="0.2032" layer="25" curve="-90"/>
+<wire x1="35.4965" y1="8.89" x2="37.1475" y2="8.89" width="0.2032" layer="25"/>
+<wire x1="37.1475" y1="8.89" x2="37.4015" y2="8.636" width="0.2032" layer="25" curve="-90"/>
+<wire x1="37.4015" y1="7.112" x2="37.1475" y2="6.858" width="0.2032" layer="25" curve="-90"/>
+<wire x1="37.1475" y1="6.858" x2="35.4965" y2="6.858" width="0.2032" layer="25"/>
+<wire x1="35.4965" y1="6.858" x2="35.2425" y2="7.112" width="0.2032" layer="25" curve="-90"/>
+<wire x1="17.526" y1="12.6365" x2="17.272" y2="12.8905" width="0.2032" layer="25" curve="-90"/>
+<wire x1="17.272" y1="12.8905" x2="17.272" y2="14.5415" width="0.2032" layer="25"/>
+<wire x1="17.272" y1="14.5415" x2="17.526" y2="14.7955" width="0.2032" layer="25" curve="-90"/>
+<wire x1="19.05" y1="14.7955" x2="19.304" y2="14.5415" width="0.2032" layer="25" curve="-90"/>
+<wire x1="19.304" y1="14.5415" x2="19.304" y2="12.8905" width="0.2032" layer="25"/>
+<wire x1="19.304" y1="12.8905" x2="19.05" y2="12.6365" width="0.2032" layer="25" curve="-90"/>
+<wire x1="12.1285" y1="14.605" x2="12.3825" y2="14.859" width="0.2032" layer="25" curve="-90"/>
+<wire x1="12.3825" y1="14.859" x2="14.0335" y2="14.859" width="0.2032" layer="25"/>
+<wire x1="14.0335" y1="14.859" x2="14.2875" y2="14.605" width="0.2032" layer="25" curve="-90"/>
+<wire x1="14.2875" y1="13.081" x2="14.0335" y2="12.827" width="0.2032" layer="25" curve="-90"/>
+<wire x1="14.0335" y1="12.827" x2="12.3825" y2="12.827" width="0.2032" layer="25"/>
+<wire x1="12.3825" y1="12.827" x2="12.1285" y2="13.081" width="0.2032" layer="24" curve="-90"/>
+<wire x1="18.161" y1="27.7495" x2="17.907" y2="28.0035" width="0.2032" layer="25" curve="-90"/>
+<wire x1="17.907" y1="28.0035" x2="17.907" y2="29.6545" width="0.2032" layer="25"/>
+<wire x1="17.907" y1="29.6545" x2="18.161" y2="29.9085" width="0.2032" layer="25" curve="-90"/>
+<wire x1="19.685" y1="29.9085" x2="19.939" y2="29.6545" width="0.2032" layer="25" curve="-90"/>
+<wire x1="19.939" y1="29.6545" x2="19.939" y2="28.0035" width="0.2032" layer="25"/>
+<wire x1="19.939" y1="28.0035" x2="19.685" y2="27.7495" width="0.2032" layer="25" curve="-90"/>
+<wire x1="16.129" y1="21.3995" x2="16.383" y2="21.6535" width="0.2032" layer="25" curve="-90"/>
+<wire x1="16.383" y1="21.6535" x2="18.034" y2="21.6535" width="0.2032" layer="25"/>
+<wire x1="18.034" y1="21.6535" x2="18.288" y2="21.3995" width="0.2032" layer="25" curve="-90"/>
+<wire x1="18.288" y1="19.8755" x2="18.034" y2="19.6215" width="0.2032" layer="25" curve="-90"/>
+<wire x1="18.034" y1="19.6215" x2="16.383" y2="19.6215" width="0.2032" layer="25"/>
+<wire x1="16.383" y1="19.6215" x2="16.129" y2="19.8755" width="0.2032" layer="25" curve="-90"/>
+<wire x1="32.1945" y1="5.7785" x2="32.1945" y2="4.3815" width="0.2032" layer="25"/>
+<wire x1="32.1945" y1="9.5885" x2="32.1945" y2="8.1915" width="0.2032" layer="25"/>
+<wire x1="32.1945" y1="2.2225" x2="32.1945" y2="0.8255" width="0.2032" layer="25"/>
+<wire x1="12.3825" y1="12.827" x2="12.1285" y2="13.081" width="0.2032" layer="25" curve="-90"/>
+<wire x1="14.732" y1="14.732" x2="14.732" y2="12.954" width="0.2032" layer="25"/>
 </plain>
 <attributes>
@@
 <attribute name="VALUE" x="16.256" y="18.9865" size="0.4064" layer="27"/>
 </element>
-<element name="R9" library="resistor" package="R0603" value="" x="14.9225" y="45.72" smashed="yes" rot="MR90">
-<attribute name="VALUE" x="12.8905" y="44.831" size="1.27" layer="28" rot="MR90"/>
+<element name="R9" library="resistor" package="R0603" value="" x="13.9065" y="45.72" smashed="yes" rot="MR90">
+<attribute name="VALUE" x="11.8745" y="44.831" size="1.27" layer="28" rot="MR90"/>
 </element>
 </elements>
@@
 <contactref element="D5" pad="1"/>
 <contactref element="R9" pad="2"/>
-<wire x1="14.92" y1="47.768" x2="14.92" y2="46.5725" width="0.381" layer="16"/>
-<wire x1="14.92" y1="46.5725" x2="14.9225" y2="46.57" width="0.381" layer="16"/>
+<wire x1="13.9065" y1="46.57" x2="14.566" y2="46.57" width="0.4064" layer="16"/>
+<wire x1="14.566" y1="46.57" x2="14.9225" y2="46.9265" width="0.4064" layer="16"/>
+<wire x1="14.9225" y1="46.9265" x2="14.9225" y2="47.7655" width="0.4064" layer="16"/>
+<wire x1="14.9225" y1="47.7655" x2="14.92" y2="47.768" width="0.4064" layer="16"/>
 </signal>
 </signals>
