File: Tilty Hardware/Board Files/Tilty Duo and Quad/V0.2.5/Eagle PCB Files/TiltyDuo.brd (EAGLE design)
At the start: 38.1 x 50.8 mm, 50 parts, among them U1 TEENSY_3.0_OUTER-PINS28-DIP_S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, U2 HC-09_BREAKOUT, U3 MPL3115A2LGA8, U4 LM2931, U5 MPU-6050, U6 HMC5883LSMD, U7 SPI_FLASH-X25XXSMD

Commit message: Lots of little changes
Parts:
- U2: value HC-09_BREAKOUT -> MPU-6050; device csr:HC-09_BREAKOUT -> SparkFun-Sensors:QFN-24
- U3: value MPL3115A2LGA8 -> LM2931; device SparkFun-Sensors:LGA8 -> on-semiconductor:TO263
- U4: value LM2931 -> SPI_FLASH-X25XXSMD; device on-semiconductor:TO263 -> SparkFun-DigitalIC:SO08
- U5: value MPU-6050 -> HC-09_BREAKOUT; device SparkFun-Sensors:QFN-24 -> csr:HC-09_BREAKOUT
- U7: value SPI_FLASH-X25XXSMD -> MPL3115A2LGA8; device SparkFun-DigitalIC:SO08 -> SparkFun-Sensors:LGA8
- moved U4 28.3 mm to (6.99, 18.9), turned to 180 degrees
- moved U7 24.5 mm to (30.0, 27.4)
- moved U3 20.3 mm to (19.1, 44.5), turned to 0 degrees
- moved U2 18.2 mm to (19.1, 25.4), turned to 90 degrees
- moved U5 18.2 mm to (22.9, 7.62), turned to 270 degrees
Connections:
- net 5V: now also U3.P$3; no longer U4.P$3
- net AUXCL: now also U2.7; no longer U5.7
- net AUXDA: now also U2.6; no longer U5.6
- net CMD: now also U5.P$34; no longer U2.P$34
- net CS: now also U4.1; no longer U7.1
- net GND: now also U2.1, U2.11, U2.18, U2.9, U3.P$1, U4.4, U5.P$13, U5.P$21, U5.P$22, U7.3; no longer U2.P$13, U2.P$21, U2.P$22, U3.3, U4.P$1, U5.1, U5.11, U5.18, U5.9, U7.4
- net MISO: now also U4.2; no longer U7.2
- net MOSI: now also U4.5; no longer U7.5
- net N$1: now also U2.10; no longer U5.10
- net N$14: now also U5.P$31; no longer U2.P$31
- net N$16: now also U2.12; no longer U5.12
- net N$2: now also U2.20; no longer U5.20
- net N$21: now also U7.2; no longer U3.2
- net RX1: now also U5.P$1; no longer U2.P$1
- net SCK: now also U4.6; no longer U7.6
- net SCL: now also U2.23, U7.8; no longer U3.8, U5.23
- net SDA: now also U2.24, U7.7; no longer U3.7, U5.24
- net TEENSY_3V3: now also U2.13, U2.8, U4.3, U4.7, U4.8, U5.P$11, U5.P$12, U7.1, U7.4; no longer U2.P$11, U2.P$12, U3.1, U3.4, U5.13, U5.8, U7.3, U7.7, U7.8
- net TX1: now also U5.P$2; no longer U2.P$2
- net VBATT: now also U3.P$2; no longer U4.P$2
- net YEL_LED: now also U5.P$32; no longer U2.P$32
