File: Tilty Hardware/Board Files/RC Receiver Adapter/V0.1.2/Eagle FIles/RC Receiver.sch (EAGLE design)
At the start: 29 parts, among them U1 ATMEGA328P, U2 LM2931, U3 AP7313SOT23R, U4 C74HC407514-SOIC, Y1 16MHz

Commit message: Added some datasheets, USB Host work
Parts:
- U3: PART# (none) -> AP7313-33SRG-7
Changed lines of the file:
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@@
 <part name="+3V1" library="supply1" deviceset="+3V3" device=""/>
 <part name="GND8" library="supply1" deviceset="GND" device=""/>
-<part name="U3" library="My Parts" deviceset="AP7313" device="SOT23R"/>
+<part name="U3" library="My Parts" deviceset="AP7313" device="SOT23R">
+<attribute name="PART#" value="AP7313-33SRG-7"/>
+</part>
 <part name="P+7" library="supply1" deviceset="+5V" device=""/>
 <part name="+3V2" library="supply1" deviceset="+3V3" device=""/>
@@
 <instance part="+3V1" gate="G$1" x="175.26" y="129.54"/>
 <instance part="GND8" gate="1" x="162.56" y="114.3"/>
-<instance part="U3" gate="G$1" x="215.9" y="101.6"/>
+<instance part="U3" gate="G$1" x="215.9" y="101.6">
+<attribute name="PART#" x="215.9" y="101.6" size="1.778" layer="96" display="off"/>
+</instance>
 <instance part="P+7" gate="1" x="198.12" y="106.68"/>
 <instance part="+3V2" gate="G$1" x="233.68" y="106.68"/>
