File: Tilty Hardware/Board Files/GPS/Eagle PCB Files/GPS adapter.brd (EAGLE design)
At the start: 38.1 x 50.8 mm, 6 parts

Commit message: GPS adapter work
Parts:
- added C1: 4.7uF, resistor:C0603
- added C2, C3: 0.1uF, resistor:C0603
- added U2: LM2931, on-semiconductor:TO263
- added U3: AP7313SOT23R, My Parts:SOT23
- renumbered U$1 to U1
Connections:
- new net N$3: C1.2, C2.2, C3.2, U2.P$1, U3.P$1
- net +3V3: now also C3.1, U3.P$2
- net +5V: now also C1.1, U2.P$3, U3.P$3
- net VCC: now also C2.1, U2.P$2
Changed lines of the file:
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@@
 <element name="JP3" library="My Parts" package="8-PIN_RECEPTACLE_LOCK_NO-SS" value="8-PIN_HEADER" x="35.56" y="20.193" rot="R270"/>
 <element name="JP4" library="My Parts" package="8-PIN_RECEPTACLE_LOCK_NO-SS" value="8-PIN_HEADER" x="30.48" y="40.513" rot="R270"/>
-<element name="U$1" library="SparkFun-RF" package="XBEE-1_LOCK" value="XBEE-1XBEE-1_LOCK" x="19.05" y="6.35"/>
+<element name="U1" library="SparkFun-RF" package="XBEE-1_LOCK" value="XBEE-1XBEE-1_LOCK" x="19.05" y="6.35"/>
 <element name="R1" library="resistor" package="R0603" value="4.7K" x="2.54" y="-3.81"/>
+<element name="U3" library="My Parts" package="SOT23" value="AP7313SOT23R" x="3.81" y="-10.16"/>
+<element name="U2" library="on-semiconductor" package="TO263" value="LM2931" x="-5.08" y="-2.54"/>
+<element name="C1" library="resistor" package="C0603" value="4.7uF" x="-6.35" y="-15.24"/>
+<element name="C2" library="resistor" package="C0603" value="0.1uF" x="-6.35" y="-19.05"/>
+<element name="C3" library="resistor" package="C0603" value="0.1uF" x="-6.35" y="-22.86"/>
 </elements>
 <signals>
@@
 <contactref element="JP3" pad="P$8"/>
 <contactref element="JP4" pad="P$2"/>
-<contactref element="U$1" pad="10"/>
+<contactref element="U1" pad="10"/>
 <wire x1="35.56" y1="11.303" x2="30.607" y2="46.863" width="0" layer="19" extent="1-1"/>
 <wire x1="8.2278" y1="8.35" x2="35.56" y2="11.303" width="0" layer="19" extent="1-1"/>
@@
 <signal name="3V_SCL">
 <contactref element="JP4" pad="P$7"/>
-<contactref element="U$1" pad="19"/>
+<contactref element="U1" pad="19"/>
 <wire x1="30.2278" y1="24.35" x2="30.353" y2="34.163" width="0" layer="19" extent="1-1"/>
 </signal>
 <signal name="3V_SDA">
 <contactref element="JP4" pad="P$8"/>
-<contactref element="U$1" pad="20"/>
+<contactref element="U1" pad="20"/>
 <wire x1="29.8722" y1="26.35" x2="30.48" y2="31.623" width="0" layer="19" extent="1-1"/>
 </signal>
 <signal name="+3V3">
 <contactref element="JP1" pad="P$1"/>
-<contactref element="U$1" pad="1"/>
+<contactref element="U1" pad="1"/>
 <contactref element="R1" pad="1"/>
+<contactref element="U3" pad="P$2"/>
+<contactref element="C3" pad="1"/>
 <wire x1="7.8722" y1="26.35" x2="7.493" y2="49.403" width="0" layer="19" extent="1-1"/>
 <wire x1="1.69" y1="-3.81" x2="7.8722" y2="26.35" width="0" layer="19" extent="1-1"/>
+<wire x1="4.76" y1="-11.31" x2="1.69" y2="-3.81" width="0" layer="19" extent="1-1"/>
+<wire x1="-7.2" y1="-22.86" x2="4.76" y2="-11.31" width="0" layer="19" extent="1-1"/>
 </signal>
 <signal name="+5V">
 <contactref element="JP4" pad="P$1"/>
+<contactref element="U2" pad="P$3"/>
+<contactref element="C1" pad="1"/>
+<contactref element="U3" pad="P$3"/>
+<wire x1="3.81" y1="-9.01" x2="30.353" y2="49.403" width="0" layer="19" extent="1-1"/>
+<wire x1="-2.794" y1="-6.9342" x2="3.81" y2="-9.01" width="0" layer="19" extent="1-1"/>
+<wire x1="-7.2" y1="-15.24" x2="-2.794" y2="-6.9342" width="0" layer="19" extent="1-1"/>
 </signal>
 <signal name="VCC">
 <contactref element="JP2" pad="P$7"/>
+<contactref element="C2" pad="1"/>
+<contactref element="U2" pad="P$2"/>
+<wire x1="-7.366" y1="-6.9342" x2="-7.2" y2="-19.05" width="0" layer="19" extent="1-1"/>
+<wire x1="2.413" y1="13.843" x2="-7.366" y2="-6.9342" width="0" layer="19" extent="1-1"/>
 </signal>
 <signal name="RX3">
-<contactref element="U$1" pad="2"/>
+<contactref element="U1" pad="2"/>
 </signal>
 <signal name="TX3">
-<contactref element="U$1" pad="3"/>
+<contactref element="U1" pad="3"/>
 </signal>
 <signal name="N$2">
-<contactref element="U$1" pad="5"/>
+<contactref element="U1" pad="5"/>
 <contactref element="R1" pad="2"/>
 <wire x1="3.39" y1="-3.81" x2="7.8722" y2="18.35" width="0" layer="19" extent="1-1"/>
 </signal>
+<signal name="N$3">
+<contactref element="U2" pad="P$1"/>
+<contactref element="U3" pad="P$1"/>
+<contactref element="C2" pad="2"/>
+<contactref element="C1" pad="2"/>
+<contactref element="C3" pad="2"/>
+<wire x1="-5.5" y1="-19.05" x2="-5.5" y2="-22.86" width="0" layer="19" extent="1-1"/>
+<wire x1="-5.5" y1="-15.24" x2="-5.5" y2="-19.05" width="0" layer="19" extent="1-1"/>
+<wire x1="2.86" y1="-11.31" x2="-5.5" y2="-15.24" width="0" layer="19" extent="1-1"/>
+<wire x1="-5.08" y1="0.254" x2="2.86" y2="-11.31" width="0" layer="19" extent="1-1"/>
+</signal>
 </signals>
