File: Tilty Hardware/Board Files/GPS/Eagle PCB Files/GPS adapter.sch (EAGLE design)
At the start: 6 parts

Commit message: GPS adapter work
Parts:
- added C1: 4.7uF, resistor:C-USC0603
- added C2, C3: 0.1uF, resistor:C-USC0603
- added U2: LM2931, on-semiconductor:LM2931
- added U3: AP7313SOT23R, My Parts:AP7313SOT23R
- renumbered U$1 to U1
Connections:
- new net N$3: C1.2, C2.2, C3.2, U2.GND, U3.GND
- net +3V3: now also C3.1, U3.VOUT
- net +5V: now also C1.1, U2.5V, U3.VIN
- net VCC: now also C2.1, U2.VIN
Changed lines of the file:
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@@
 <part name="P+1" library="supply1" deviceset="+5V" device=""/>
 <part name="P+2" library="supply1" deviceset="VCC" device=""/>
-<part name="U$1" library="SparkFun-RF" deviceset="XBEE-1" device="XBEE-1_LOCK"/>
+<part name="U1" library="SparkFun-RF" deviceset="XBEE-1" device="XBEE-1_LOCK"/>
 <part name="+3V2" library="supply1" deviceset="+3V3" device=""/>
 <part name="GND1" library="supply1" deviceset="GND" device=""/>
 <part name="+3V3" library="supply1" deviceset="+3V3" device=""/>
 <part name="R1" library="resistor" deviceset="R-US_" device="R0603" value="4.7K"/>
+<part name="U3" library="My Parts" deviceset="AP7313" device="SOT23R"/>
+<part name="U2" library="on-semiconductor" deviceset="LM2931" device=""/>
+<part name="C1" library="resistor" deviceset="C-US" device="C0603" value="4.7uF"/>
+<part name="C2" library="resistor" deviceset="C-US" device="C0603" value="0.1uF"/>
+<part name="C3" library="resistor" deviceset="C-US" device="C0603" value="0.1uF"/>
+<part name="P+3" library="supply1" deviceset="+5V" device=""/>
+<part name="+3V4" library="supply1" deviceset="+3V3" device=""/>
+<part name="P+4" library="supply1" deviceset="VCC" device=""/>
 </parts>
 <sheets>
@@
 <instance part="P+1" gate="1" x="25.4" y="27.94"/>
 <instance part="P+2" gate="VCC" x="30.48" y="66.04"/>
-<instance part="U$1" gate="G$1" x="99.06" y="66.04"/>
+<instance part="U1" gate="G$1" x="99.06" y="66.04"/>
 <instance part="+3V2" gate="G$1" x="76.2" y="83.82"/>
 <instance part="GND1" gate="1" x="76.2" y="48.26"/>
 <instance part="+3V3" gate="G$1" x="66.04" y="71.12"/>
 <instance part="R1" gate="G$1" x="73.66" y="66.04"/>
+<instance part="U3" gate="G$1" x="96.52" y="15.24"/>
+<instance part="U2" gate="G$1" x="60.96" y="12.7" smashed="yes">
+<attribute name="NAME" x="55.88" y="19.05" size="2.54" layer="95"/>
+</instance>
+<instance part="C1" gate="G$1" x="76.2" y="10.16"/>
+<instance part="C2" gate="G$1" x="40.64" y="10.16"/>
+<instance part="C3" gate="G$1" x="111.76" y="10.16"/>
+<instance part="P+3" gate="1" x="78.74" y="20.32"/>
+<instance part="+3V4" gate="G$1" x="114.3" y="20.32"/>
+<instance part="P+4" gate="VCC" x="40.64" y="20.32"/>
 </instances>
 <busses>
@@
 </segment>
 <segment>
-<pinref part="U$1" gate="G$1" pin="GND"/>
+<pinref part="U1" gate="G$1" pin="GND"/>
 <wire x1="78.74" y1="53.34" x2="76.2" y2="53.34" width="0.1524" layer="91"/>
 <wire x1="76.2" y1="53.34" x2="76.2" y2="50.8" width="0.1524" layer="91"/>
@@
 </segment>
 <segment>
-<pinref part="U$1" gate="G$1" pin="DIO1"/>
+<pinref part="U1" gate="G$1" pin="DIO1"/>
 <wire x1="119.38" y1="73.66" x2="132.08" y2="73.66" width="0.1524" layer="91"/>
 <label x="121.92" y="73.66" size="1.778" layer="95"/>
@@
 </segment>
 <segment>
-<pinref part="U$1" gate="G$1" pin="DIO0"/>
+<pinref part="U1" gate="G$1" pin="DIO0"/>
 <wire x1="119.38" y1="76.2" x2="132.08" y2="76.2" width="0.1524" layer="91"/>
 <label x="121.92" y="76.2" size="1.778" layer="95"/>
@@
 </segment>
 <segment>
-<pinref part="U$1" gate="G$1" pin="VDD"/>
+<pinref part="U1" gate="G$1" pin="VDD"/>
 <wire x1="78.74" y1="76.2" x2="76.2" y2="76.2" width="0.1524" layer="91"/>
 <wire x1="76.2" y1="76.2" x2="76.2" y2="81.28" width="0.1524" layer="91"/>
@@
 <wire x1="66.04" y1="66.04" x2="68.58" y2="66.04" width="0.1524" layer="91"/>
 </segment>
+<segment>
+<pinref part="+3V4" gate="G$1" pin="+3V3"/>
+<wire x1="114.3" y1="17.78" x2="114.3" y2="15.24" width="0.1524" layer="91"/>
+<pinref part="U3" gate="G$1" pin="VOUT"/>
+<pinref part="C3" gate="G$1" pin="1"/>
+<wire x1="111.76" y1="12.7" x2="111.76" y2="15.24" width="0.1524" layer="91"/>
+<wire x1="114.3" y1="15.24" x2="111.76" y2="15.24" width="0.1524" layer="91"/>
+<junction x="111.76" y="15.24"/>
+</segment>
 </net>
 <net name="+5V" class="0">
@@
 <wire x1="25.4" y1="20.32" x2="25.4" y2="25.4" width="0.1524" layer="91"/>
 </segment>
+<segment>
+<pinref part="U2" gate="G$1" pin="5V"/>
+<pinref part="C1" gate="G$1" pin="1"/>
+<wire x1="76.2" y1="15.24" x2="76.2" y2="12.7" width="0.1524" layer="91"/>
+<pinref part="U3" gate="G$1" pin="VIN"/>
+<wire x1="76.2" y1="15.24" x2="78.74" y2="15.24" width="0.1524" layer="91"/>
+<junction x="76.2" y="15.24"/>
+<pinref part="P+3" gate="1" pin="+5V"/>
+<wire x1="78.74" y1="15.24" x2="81.28" y2="15.24" width="0.1524" layer="91"/>
+<wire x1="78.74" y1="17.78" x2="78.74" y2="15.24" width="0.1524" layer="91"/>
+<junction x="78.74" y="15.24"/>
+</segment>
 </net>
 <net name="VCC" class="0">
@@
 <wire x1="30.48" y1="60.96" x2="30.48" y2="63.5" width="0.1524" layer="91"/>
 </segment>
+<segment>
+<pinref part="C2" gate="G$1" pin="1"/>
+<wire x1="40.64" y1="12.7" x2="40.64" y2="15.24" width="0.1524" layer="91"/>
+<pinref part="U2" gate="G$1" pin="VIN"/>
+<wire x1="40.64" y1="15.24" x2="45.72" y2="15.24" width="0.1524" layer="91"/>
+<pinref part="P+4" gate="VCC" pin="VCC"/>
+<wire x1="40.64" y1="17.78" x2="40.64" y2="15.24" width="0.1524" layer="91"/>
+<junction x="40.64" y="15.24"/>
+</segment>
 </net>
 <net name="RX3" class="0">
 <segment>
-<pinref part="U$1" gate="G$1" pin="DOUT"/>
+<pinref part="U1" gate="G$1" pin="DOUT"/>
 <wire x1="78.74" y1="73.66" x2="71.12" y2="73.66" width="0.1524" layer="91"/>
 <label x="71.12" y="73.66" size="1.778" layer="95"/>
@@
 <net name="TX3" class="0">
 <segment>
-<pinref part="U$1" gate="G$1" pin="DIN"/>
+<pinref part="U1" gate="G$1" pin="DIN"/>
 <wire x1="78.74" y1="71.12" x2="71.12" y2="71.12" width="0.1524" layer="91"/>
 <label x="71.12" y="71.12" size="1.778" layer="95"/>
@@
 <net name="N$2" class="0">
 <segment>
-<pinref part="U$1" gate="G$1" pin="RESET"/>
+<pinref part="U1" gate="G$1" pin="RESET"/>
 <pinref part="R1" gate="G$1" pin="2"/>
 </segment>
 </net>
+<net name="N$3" class="0">
+<segment>
+<pinref part="U2" gate="G$1" pin="GND"/>
+<pinref part="U3" gate="G$1" pin="GND"/>
+<wire x1="60.96" y1="2.54" x2="76.2" y2="2.54" width="0.1524" layer="91"/>
+<pinref part="C2" gate="G$1" pin="2"/>
+<wire x1="76.2" y1="2.54" x2="96.52" y2="2.54" width="0.1524" layer="91"/>
+<wire x1="40.64" y1="5.08" x2="40.64" y2="2.54" width="0.1524" layer="91"/>
+<wire x1="40.64" y1="2.54" x2="60.96" y2="2.54" width="0.1524" layer="91"/>
+<junction x="60.96" y="2.54"/>
+<pinref part="C1" gate="G$1" pin="2"/>
+<wire x1="76.2" y1="5.08" x2="76.2" y2="2.54" width="0.1524" layer="91"/>
+<junction x="76.2" y="2.54"/>
+<pinref part="C3" gate="G$1" pin="2"/>
+<wire x1="96.52" y1="2.54" x2="111.76" y2="2.54" width="0.1524" layer="91"/>
+<wire x1="111.76" y1="2.54" x2="111.76" y2="5.08" width="0.1524" layer="91"/>
+<junction x="96.52" y="2.54"/>
+</segment>
+</net>
