File: Tilty Hardware/Board Files/Tilty Template/Eagle PCB Files/Tilty Template.brd (EAGLE design)
At the start: 38.1 x 50.8 mm, 4 parts

Commit message: Ordered USB Host add-on prototype
Added folder for next revision and updated Tilty Template to show
reserved pins
Connections:
- net N$10 renamed USB_CS
Changed lines of the file:
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@@
 <contactref element="JP1" pad="P$7"/>
 </signal>
-<signal name="N$10">
+<signal name="USB_CS">
 <contactref element="JP1" pad="P$6"/>
 </signal>
