File: Tilty Hardware/Board Files/Tilty Template/Eagle PCB Files/Tilty Template.sch (EAGLE design)
At the start: 4 parts

Commit message: Ordered USB Host add-on prototype
Added folder for next revision and updated Tilty Template to show
reserved pins
Connections:
- net N$10 renamed USB_CS
Other:
- note added: "<-used by add-on"
Changed lines of the file:
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@@
 <text x="-3.175" y="98.044" size="1.778" layer="91" ratio="15">*</text>
 <text x="-3.175" y="100.584" size="1.778" layer="91" ratio="15">*</text>
+<text x="25.4" y="91.44" size="1.778" layer="91">&lt;-used by add-on</text>
 </plain>
 <instances>
@@
 </segment>
 </net>
-<net name="N$10" class="0">
+<net name="USB_CS" class="0">
 <segment>
 <pinref part="JP1" gate="G$1" pin="6"/>
 <wire x1="5.08" y1="91.44" x2="25.4" y2="91.44" width="0.1524" layer="91"/>
+<label x="15.24" y="91.44" size="1.778" layer="95"/>
 </segment>
 </net>
