File: Tilty Hardware/Board Files/USB Host/V0.1.0/Eagle PCB Files/USB Host.brd (EAGLE design)
At the start: 38.1 x 50.8 mm, 24 parts, among them U1 MAX3421E, U2 AP7313SOT23R, U3 LM2931

Commit message: A bunch of changes to things.todo after assembling new prototypes
Parts:
- C6: value 1uF -> 0.1uF
Changed lines of the file:
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@@
 </element>
 <element name="U2" library="My Parts" package="SOT23" value="AP7313SOT23R" x="18.034" y="30.48" smashed="yes"/>
-<element name="C6" library="resistor" package="C0603" value="1uF" x="17.9705" y="27.94" smashed="yes" rot="R180">
+<element name="C6" library="resistor" package="C0603" value="0.1uF" x="17.9705" y="27.94" smashed="yes" rot="R180">
 <attribute name="VALUE" x="18.8595" y="29.972" size="1.27" layer="27" rot="R180"/>
 </element>
