File: Tilty Hardware/Board Files/USB Host/V0.1.0/Eagle PCB Files/USB Host.sch (EAGLE design)
At the start: 24 parts, among them U1 MAX3421E, U2 AP7313SOT23R, U3 LM2931

Commit message: A bunch of changes to things.todo after assembling new prototypes
Parts:
- C6: value 1uF -> 0.1uF
Changed lines of the file:
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@@
 <part name="C5" library="resistor" deviceset="C-US" device="C0603" value="4.7uF"/>
 <part name="U2" library="My Parts" deviceset="AP7313" device="SOT23R"/>
-<part name="C6" library="resistor" deviceset="C-US" device="C0603" value="1uF"/>
+<part name="C6" library="resistor" deviceset="C-US" device="C0603" value="0.1uF"/>
 <part name="U3" library="on-semiconductor" deviceset="LM2931" device=""/>
 <part name="C7" library="resistor" deviceset="C-US" device="C0603" value="0.1uF"/>
