File: Tilty Hardware/Board Files/USB Host/V0.1.1/Eagle PCB Files/USB Host.sch (EAGLE design)
At the start: 24 parts, among them U1 MAX3421E, U2 AP7313SOT23R, U3 LM2931

Commit message: A bunch of changes to things.todo after assembling new prototypes
Connections:
- removed net N$27: JP4.6
- net INT: now also JP4.6
Changed lines of the file:
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@@
-</segment>
-</net>
-<net name="N$27" class="0">
-<segment>
-<pinref part="JP4" gate="G$1" pin="6"/>
-<wire x1="5.08" y1="7.62" x2="22.86" y2="7.62" width="0.1524" layer="91"/>
 </segment>
 </net>
@@
 <pinref part="R3" gate="G$1" pin="1"/>
 </segment>
-</net>
+<segment>
+<pinref part="JP4" gate="G$1" pin="6"/>
+<wire x1="5.08" y1="7.62" x2="22.86" y2="7.62" width="0.1524" layer="91"/>
+</segment>
+</net>

Commit message: Added Tilty silkscreen and option 5/3.3v I2C connections
Parts:
- removed C1: 0.1uF, resistor:C-USC0603
Connections:
- net +3V3: no longer C1.1
- net GND: no longer C1.2
Other:
- moved on the sheet: C2
Changed lines of the file:
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@@
 <part name="GND1" library="supply1" deviceset="GND" device=""/>
 <part name="GND2" library="supply1" deviceset="GND" device=""/>
-<part name="C1" library="resistor" deviceset="C-US" device="C0603" value="0.1uF"/>
 <part name="C2" library="resistor" deviceset="C-US" device="C0603" value="0.1uF"/>
 <part name="GND3" library="supply1" deviceset="GND" device=""/>
@@
 <instance part="GND1" gate="1" x="76.2" y="35.56"/>
 <instance part="GND2" gate="1" x="124.46" y="5.08"/>
-<instance part="C1" gate="G$1" x="101.6" y="78.74"/>
-<instance part="C2" gate="G$1" x="88.9" y="78.74"/>
-<instance part="GND3" gate="1" x="88.9" y="66.04"/>
+<instance part="C2" gate="G$1" x="101.6" y="78.74"/>
+<instance part="GND3" gate="1" x="101.6" y="68.58"/>
 <instance part="P+3" gate="1" x="83.82" y="63.5"/>
 <instance part="X1" gate="G$1" x="93.98" y="25.4" rot="R90">
@@
 <segment>
 <pinref part="C2" gate="G$1" pin="2"/>
-<wire x1="88.9" y1="73.66" x2="88.9" y2="71.12" width="0.1524" layer="91"/>
-<pinref part="C1" gate="G$1" pin="2"/>
-<wire x1="88.9" y1="71.12" x2="101.6" y2="71.12" width="0.1524" layer="91"/>
-<wire x1="101.6" y1="71.12" x2="101.6" y2="73.66" width="0.1524" layer="91"/>
 <pinref part="GND3" gate="1" pin="GND"/>
-<wire x1="88.9" y1="71.12" x2="88.9" y2="68.58" width="0.1524" layer="91"/>
-<junction x="88.9" y="71.12"/>
+<wire x1="101.6" y1="73.66" x2="101.6" y2="71.12" width="0.1524" layer="91"/>
 </segment>
 <segment>
@@
 <segment>
 <pinref part="C2" gate="G$1" pin="1"/>
-<wire x1="88.9" y1="81.28" x2="88.9" y2="83.82" width="0.1524" layer="91"/>
-<pinref part="C1" gate="G$1" pin="1"/>
-<wire x1="88.9" y1="83.82" x2="101.6" y2="83.82" width="0.1524" layer="91"/>
-<wire x1="101.6" y1="83.82" x2="101.6" y2="81.28" width="0.1524" layer="91"/>
+<wire x1="101.6" y1="81.28" x2="101.6" y2="83.82" width="0.1524" layer="91"/>
+<wire x1="101.6" y1="83.82" x2="111.76" y2="83.82" width="0.1524" layer="91"/>
 <pinref part="U1" gate="G$1" pin="VCC"/>
-<wire x1="101.6" y1="83.82" x2="111.76" y2="83.82" width="0.1524" layer="91"/>
 <wire x1="111.76" y1="83.82" x2="111.76" y2="73.66" width="0.1524" layer="91"/>
-<junction x="101.6" y="83.82"/>
 <pinref part="U1" gate="G$1" pin="VL"/>
 <wire x1="111.76" y1="73.66" x2="119.38" y2="73.66" width="0.1524" layer="91"/>
@@
 <pinref part="JP4" gate="G$1" pin="6"/>
 <wire x1="5.08" y1="7.62" x2="22.86" y2="7.62" width="0.1524" layer="91"/>
-</segment>
-</net>
+<label x="10.16" y="7.62" size="1.778" layer="95"/>
+</segment>
+</net>

Commit message: Added reset pullup to USB Host add-on
Oops... That should've been there before...
Parts:
- added R5: 10K, resistor:R-US_R0603
- R3: value 4.7K -> 10K
Connections:
- net +3V3: now also R5.2
- net RST: now also R5.1
Changed lines of the file:
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@@
 <part name="R1" library="resistor" deviceset="R-US_" device="R0603" value="33"/>
 <part name="R2" library="resistor" deviceset="R-US_" device="R0603" value="33"/>
-<part name="R3" library="resistor" deviceset="R-US_" device="R0603" value="4.7K"/>
+<part name="R3" library="resistor" deviceset="R-US_" device="R0603" value="10K"/>
 <part name="GND1" library="supply1" deviceset="GND" device=""/>
 <part name="GND2" library="supply1" deviceset="GND" device=""/>
@@
 <part name="P+7" library="supply1" deviceset="+5V" device=""/>
 <part name="GND8" library="supply1" deviceset="GND" device=""/>
+<part name="R5" library="resistor" deviceset="R-US_" device="R0603" value="10K"/>
 </parts>
 <sheets>
@@
 <instance part="P+7" gate="1" x="38.1" y="81.28"/>
 <instance part="GND8" gate="1" x="60.96" y="71.12"/>
+<instance part="R5" gate="G$1" x="116.84" y="81.28" rot="R180"/>
 </instances>
 <busses>
@@
 <wire x1="101.6" y1="83.82" x2="111.76" y2="83.82" width="0.1524" layer="91"/>
 <pinref part="U1" gate="G$1" pin="VCC"/>
-<wire x1="111.76" y1="83.82" x2="111.76" y2="73.66" width="0.1524" layer="91"/>
+<wire x1="111.76" y1="83.82" x2="111.76" y2="81.28" width="0.1524" layer="91"/>
 <pinref part="U1" gate="G$1" pin="VL"/>
+<wire x1="111.76" y1="81.28" x2="111.76" y2="73.66" width="0.1524" layer="91"/>
 <wire x1="111.76" y1="73.66" x2="119.38" y2="73.66" width="0.1524" layer="91"/>
 <junction x="111.76" y="73.66"/>
@@
 <wire x1="116.84" y1="86.36" x2="111.76" y2="86.36" width="0.1524" layer="91"/>
 <junction x="111.76" y="86.36"/>
+<pinref part="R5" gate="G$1" pin="2"/>
+<junction x="111.76" y="81.28"/>
 </segment>
 <segment>
@@
 <wire x1="124.46" y1="73.66" x2="124.46" y2="81.28" width="0.1524" layer="91"/>
 <label x="124.46" y="76.2" size="1.778" layer="95" rot="R90"/>
-</segment>
-</net>
+<pinref part="R5" gate="G$1" pin="1"/>
+<wire x1="121.92" y1="81.28" x2="124.46" y2="81.28" width="0.1524" layer="91"/>
+</segment>
+</net>

Commit message: USB Host add-on work
Parts:
- added SJ1: SOLDERJUMPERTRACE, SparkFun-Passives:SOLDERJUMPERTRACE
Connections:
- new net INT_PIN: R3.1, SJ1.2, U1.INT
- net INT: now also SJ1.1; no longer R3.1, U1.INT
Changed lines of the file:
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@@
 <part name="GND8" library="supply1" deviceset="GND" device=""/>
 <part name="R5" library="resistor" deviceset="R-US_" device="R0603" value="10K"/>
+<part name="SJ1" library="SparkFun-Passives" deviceset="SOLDERJUMPER" device="TRACE"/>
 </parts>
 <sheets>
@@
 <instance part="GND8" gate="1" x="60.96" y="71.12"/>
 <instance part="R5" gate="G$1" x="116.84" y="81.28" rot="R180"/>
+<instance part="SJ1" gate="1" x="119.38" y="99.06" smashed="yes">
+<attribute name="NAME" x="116.84" y="101.6" size="1.778" layer="95"/>
+</instance>
 </instances>
 <busses>
@@
 <net name="INT" class="0">
 <segment>
-<pinref part="U1" gate="G$1" pin="INT"/>
-<wire x1="127" y1="73.66" x2="127" y2="86.36" width="0.1524" layer="91"/>
-<label x="127" y="78.74" size="1.778" layer="95" rot="R90"/>
-<pinref part="R3" gate="G$1" pin="1"/>
-</segment>
-<segment>
 <pinref part="JP4" gate="G$1" pin="6"/>
 <wire x1="5.08" y1="7.62" x2="22.86" y2="7.62" width="0.1524" layer="91"/>
 <label x="10.16" y="7.62" size="1.778" layer="95"/>
+</segment>
+<segment>
+<pinref part="SJ1" gate="1" pin="1"/>
+<wire x1="114.3" y1="99.06" x2="109.22" y2="99.06" width="0.1524" layer="91"/>
+<label x="109.22" y="99.06" size="1.778" layer="95"/>
 </segment>
 </net>
@@
 </segment>
 </net>
+<net name="INT_PIN" class="0">
+<segment>
+<pinref part="U1" gate="G$1" pin="INT"/>
+<wire x1="127" y1="73.66" x2="127" y2="86.36" width="0.1524" layer="91"/>
+<pinref part="R3" gate="G$1" pin="1"/>
+<wire x1="127" y1="86.36" x2="127" y2="99.06" width="0.1524" layer="91"/>
+<junction x="127" y="86.36"/>
+<pinref part="SJ1" gate="1" pin="2"/>
+<wire x1="127" y1="99.06" x2="124.46" y2="99.06" width="0.1524" layer="91"/>
+</segment>
+</net>
