File: Tilty Hardware/Board Files/USB Host/V0.1.1/Eagle PCB Files/USB Host.sch (EAGLE design)
At the start: 25 parts, among them U1 MAX3421E, U2 AP7313SOT23R, U3 LM2931

Commit message: Altered USB host interrupt solderpad
Connections:
- removed net INT_PIN: R3.1, SJ1.2, U1.INT
- new net N$10: SJ1.1, U1.INT
- net INT: now also R3.1, SJ1.2; no longer SJ1.1
Changed lines of the file:
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@@
 <instance part="GND8" gate="1" x="60.96" y="71.12"/>
 <instance part="R5" gate="G$1" x="116.84" y="81.28" rot="R180"/>
-<instance part="SJ1" gate="1" x="119.38" y="99.06" smashed="yes">
-<attribute name="NAME" x="116.84" y="101.6" size="1.778" layer="95"/>
-</instance>
+<instance part="SJ1" gate="1" x="127" y="78.74" smashed="yes" rot="R90"/>
 </instances>
 <busses>
@@
 </segment>
 <segment>
-<pinref part="SJ1" gate="1" pin="1"/>
-<wire x1="114.3" y1="99.06" x2="109.22" y2="99.06" width="0.1524" layer="91"/>
-<label x="109.22" y="99.06" size="1.778" layer="95"/>
+<pinref part="SJ1" gate="1" pin="2"/>
+<pinref part="R3" gate="G$1" pin="1"/>
+<wire x1="127" y1="83.82" x2="127" y2="86.36" width="0.1524" layer="91"/>
+<wire x1="127" y1="86.36" x2="127" y2="93.98" width="0.1524" layer="91"/>
+<wire x1="127" y1="93.98" x2="119.38" y2="93.98" width="0.1524" layer="91"/>
+<junction x="127" y="86.36"/>
+<label x="119.38" y="93.98" size="1.778" layer="95"/>
 </segment>
 </net>
@@
 </segment>
 </net>
-<net name="INT_PIN" class="0">
+<net name="N$10" class="0">
 <segment>
 <pinref part="U1" gate="G$1" pin="INT"/>
-<wire x1="127" y1="73.66" x2="127" y2="86.36" width="0.1524" layer="91"/>
-<pinref part="R3" gate="G$1" pin="1"/>
-<wire x1="127" y1="86.36" x2="127" y2="99.06" width="0.1524" layer="91"/>
-<junction x="127" y="86.36"/>
-<pinref part="SJ1" gate="1" pin="2"/>
-<wire x1="127" y1="99.06" x2="124.46" y2="99.06" width="0.1524" layer="91"/>
-</segment>
-</net>
+<pinref part="SJ1" gate="1" pin="1"/>
+</segment>
+</net>

Commit message: LOTS of cleaning house....
Parts:
- C6: value 1uF -> ).F
- X1: value (none) -> 12MHz
Changed lines of the file:
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@@
 <part name="GND3" library="supply1" deviceset="GND" device=""/>
 <part name="P+3" library="supply1" deviceset="+5V" device=""/>
-<part name="X1" library="SparkFun-FreqCtrl" deviceset="CRYSTAL" device="TXC-7A">
+<part name="X1" library="SparkFun-FreqCtrl" deviceset="CRYSTAL" device="TXC-7A" value="12MHz">
 <attribute name="PART#" value="7A-12.000MAAE-T"/>
 </part>
@@
 <part name="C5" library="resistor" deviceset="C-US" device="C0603" value="4.7uF"/>
 <part name="U2" library="My Parts" deviceset="AP7313" device="SOT23R"/>
-<part name="C6" library="resistor" deviceset="C-US" device="C0603" value="1uF"/>
+<part name="C6" library="resistor" deviceset="C-US" device="C0603" value=").F"/>
 <part name="U3" library="on-semiconductor" deviceset="LM2931" device=""/>
 <part name="C7" library="resistor" deviceset="C-US" device="C0603" value="0.1uF"/>
