File: Tilty Hardware/Board Files/Dual Motor Driver/V0.1.4/Eagle PCB Files/Dual Motor Driver.sch (EAGLE design)
At the start: 42 parts, among them J1 AVR_SPI_PRG_62X3_LOCK, Q1 16MHz, U1 ATMEGA328P, U2 L298_BRIDGE_DRIVER, U3 LM2931

Commit message: Updated Dual Motor Driver to (hopefully) final revision
Parts:
- removed S1: SWITCH-MOMENTARY-2SMD, SparkFun-Electromechanical:SWITCH-MOMENTARY-2SMD
- JP8: device SparkFun-Connectors:M04LOCK -> SparkFun-Connectors:M05PTH
Connections:
- net GND: no longer S1.1
- net RESET: now also JP8.5; no longer S1.2
Changed lines of the file:
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@@
 <part name="C8" library="resistor" deviceset="C-US" device="C0603" value="22pF"/>
 <part name="GND12" library="supply1" deviceset="GND" device=""/>
-<part name="GND8" library="supply1" deviceset="GND" device=""/>
-<part name="S1" library="SparkFun-Electromechanical" deviceset="SWITCH-MOMENTARY-2" device="SMD"/>
 <part name="U1" library="SparkFun-DigitalIC" deviceset="ATMEGA328_SMT" device="" value="ATMEGA328P"/>
 <part name="GND2" library="supply1" deviceset="GND" device=""/>
@@
 <part name="U3" library="on-semiconductor" deviceset="LM2931" device=""/>
 <part name="GND14" library="supply1" deviceset="GND" device=""/>
-<part name="JP8" library="SparkFun-Connectors" deviceset="M04" device="LOCK"/>
+<part name="JP8" library="SparkFun-Connectors" deviceset="M05" device="PTH"/>
 <part name="P+10" library="supply1" deviceset="+5V" device=""/>
 <part name="GND15" library="supply1" deviceset="GND" device=""/>
@@
 <instance part="C8" gate="G$1" x="7.62" y="45.72" rot="R90"/>
 <instance part="GND12" gate="1" x="-2.54" y="38.1"/>
-<instance part="GND8" gate="1" x="12.7" y="63.5"/>
-<instance part="S1" gate="G$1" x="17.78" y="68.58" smashed="yes">
-<attribute name="NAME" x="15.24" y="71.12" size="1.778" layer="95"/>
-</instance>
 <instance part="U1" gate="G$1" x="48.26" y="43.18"/>
 <instance part="GND2" gate="1" x="22.86" y="7.62"/>
@@
 <instance part="U3" gate="G$1" x="187.96" y="73.66"/>
 <instance part="GND14" gate="1" x="71.12" y="129.54" rot="R180"/>
-<instance part="JP8" gate="G$1" x="114.3" y="48.26" rot="MR180"/>
+<instance part="JP8" gate="G$1" x="114.3" y="45.72" rot="MR180"/>
 <instance part="P+10" gate="1" x="121.92" y="58.42"/>
-<instance part="GND15" gate="1" x="127" y="43.18"/>
+<instance part="GND15" gate="1" x="129.54" y="43.18"/>
 <instance part="JP9" gate="G$1" x="111.76" y="78.74"/>
 <instance part="JP10" gate="G$1" x="111.76" y="66.04"/>
@@
 </segment>
 <segment>
-<pinref part="GND8" gate="1" pin="GND"/>
-<pinref part="S1" gate="G$1" pin="1"/>
-<wire x1="12.7" y1="68.58" x2="12.7" y2="66.04" width="0.1524" layer="91"/>
-</segment>
-<segment>
 <pinref part="GND2" gate="1" pin="GND"/>
 <pinref part="U1" gate="G$1" pin="GND@2"/>
@@
 <pinref part="JP8" gate="G$1" pin="2"/>
 <pinref part="GND15" gate="1" pin="GND"/>
-<wire x1="119.38" y1="48.26" x2="127" y2="48.26" width="0.1524" layer="91"/>
-<wire x1="127" y1="48.26" x2="127" y2="45.72" width="0.1524" layer="91"/>
+<wire x1="121.92" y1="48.26" x2="129.54" y2="48.26" width="0.1524" layer="91"/>
+<wire x1="129.54" y1="48.26" x2="129.54" y2="45.72" width="0.1524" layer="91"/>
 </segment>
 <segment>
@@
 <pinref part="JP8" gate="G$1" pin="1"/>
 <pinref part="P+10" gate="1" pin="+5V"/>
-<wire x1="119.38" y1="50.8" x2="121.92" y2="50.8" width="0.1524" layer="91"/>
 <wire x1="121.92" y1="50.8" x2="121.92" y2="55.88" width="0.1524" layer="91"/>
 </segment>
@@
 <wire x1="22.86" y1="71.12" x2="22.86" y2="68.58" width="0.1524" layer="91"/>
 <wire x1="22.86" y1="68.58" x2="25.4" y2="68.58" width="0.1524" layer="91"/>
-<pinref part="S1" gate="G$1" pin="2"/>
+<wire x1="22.86" y1="68.58" x2="10.16" y2="68.58" width="0.1524" layer="91"/>
 <junction x="22.86" y="68.58"/>
+<label x="10.16" y="68.58" size="1.778" layer="95"/>
+</segment>
+<segment>
+<pinref part="JP8" gate="G$1" pin="5"/>
+<wire x1="121.92" y1="40.64" x2="121.92" y2="35.56" width="0.1524" layer="91"/>
+<wire x1="121.92" y1="35.56" x2="132.08" y2="35.56" width="0.1524" layer="91"/>
+<label x="124.46" y="35.56" size="1.778" layer="95"/>
 </segment>
 </net>
@@
 <segment>
 <pinref part="JP8" gate="G$1" pin="3"/>
-<wire x1="119.38" y1="45.72" x2="124.46" y2="45.72" width="0.1524" layer="91"/>
+<wire x1="121.92" y1="45.72" x2="124.46" y2="45.72" width="0.1524" layer="91"/>
 <label x="121.92" y="45.72" size="1.778" layer="95"/>
 </segment>
@@
 <segment>
 <pinref part="JP8" gate="G$1" pin="4"/>
-<wire x1="119.38" y1="43.18" x2="124.46" y2="43.18" width="0.1524" layer="91"/>
+<wire x1="121.92" y1="43.18" x2="124.46" y2="43.18" width="0.1524" layer="91"/>
 <label x="121.92" y="43.18" size="1.778" layer="95"/>
 </segment>
