File: Tilty Hardware/Board Files/Dual Motor Driver/V0.1.4 with programming/Eagle PCB Files/Dual Motor Driver.sch (EAGLE design)
At the start: 43 parts, among them J1 AVR_SPI_PRG_62X3_LOCK, Q1 16MHz, U1 ATMEGA328P, U2 L298_BRIDGE_DRIVER, U3 LM2931

Commit message: Nicely laid out Dual Motor Driver with programming capability
Other:
- note added: "Headers can connect Tilty pin 0 to Reset and programming pins are connected to SPI pins"
Changed lines of the file:
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@@
 <sheet>
 <plain>
+<text x="187.96" y="0" size="1.778" layer="91">Headers can connect Tilty pin 0
+to Reset and programming pins
+are connected to SPI pins</text>
 </plain>
 <instances>
@@
 </schematic>
 </drawing>
+<compatibility>
+<note version="6.3" minversion="6.2.2" severity="warning">
+Since Version 6.2.2 text objects can contain more than one line,
+which will not be processed correctly with this version.
+</note>
+</compatibility>
 </eagle>
