File: Tilty Hardware/Board Files/Dual Motor Driver/V1.0.0/Eagle PCB Files/Dual Motor Driver.brd (EAGLE design)
At the start: 38.4 x 50.8 mm, 43 parts, among them J1 AVR_SPI_PRG_62X3_LOCK, Q1 16MHz, U1 ATMEGA328P, U2 L298_BRIDGE_DRIVER, U3 LM2931

Commit message: Updated some pin connection names on the Dual Motor Driver schematic
Connections:
- net ENC1A: now also JP5.P$3, U1.23; no longer JP6.P$3, U1.32
- net ENC1B: now also JP5.P$5, U1.1; no longer JP6.P$5, U1.24
- net ENC2A: now also JP6.P$3, U1.32; no longer JP5.P$3, U1.23
- net ENC2B: now also JP6.P$5, U1.24; no longer JP5.P$5, U1.1
- net M1+: now also U1.11, U2.13; no longer U1.2, U2.7
- net M1-: now also U1.12, U2.15; no longer U1.13, U2.9
- net M1A: now also D3.1, D6.2, JP10.2, JP5.P$1, U2.16; no longer D1.1, D8.2, JP6.P$1, JP9.2, U2.4
- net M1B: now also D4.1, D5.2, JP10.1, JP5.P$2, U2.17; no longer D2.1, D7.2, JP6.P$2, JP9.1, U2.5
- net M2+: now also U1.2, U2.7; no longer U1.11, U2.13
- net M2-: now also U1.13, U2.9; no longer U1.12, U2.15
- net M2A: now also D1.1, D8.2, JP6.P$1, JP9.2, U2.4; no longer D3.1, D6.2, JP10.2, JP5.P$1, U2.16
- net M2B: now also D2.1, D7.2, JP6.P$2, JP9.1, U2.5; no longer D4.1, D5.2, JP10.1, JP5.P$2, U2.17
- net PWM1: now also U1.9, U2.14; no longer U1.10, U2.8
- net PWM2: now also U1.10, U2.8; no longer U1.9, U2.14
- net SENSE_1: now also R4.2, R5.2, U1.26, U2.19; no longer R2.2, R3.2, U1.25, U2.2
- net SENSE_2: now also R2.2, R3.2, U1.25, U2.2; no longer R4.2, R5.2, U1.26, U2.19
Routing:
- net M2+: track 16.0 -> 30.1 mm, vias 0 -> 2
- net M1+: track 30.1 -> 16.0 mm, vias 2 -> 0
- net M2B: track 35.7 -> 44.6 mm, vias 0 -> 1
- net M1B: track 44.6 -> 35.7 mm, vias 1 -> 0
- net M2A: track 42.6 -> 37.0 mm, vias 1 -> 0
- net M1A: track 37.0 -> 42.6 mm, vias 0 -> 1
- net ENC2A: track 28.6 -> 24.0 mm
- net ENC1A: track 24.0 -> 28.6 mm
- net SENSE_2: track 39.6 -> 35.6 mm
- net SENSE_1: track 35.6 -> 39.6 mm
- net PWM2: track 16.2 -> 20.2 mm
- net PWM1: track 20.2 -> 16.2 mm
- net M2-: track 19.3 -> 16.0 mm
- net M1-: track 16.0 -> 19.3 mm
- net ENC2B: track 16.5 -> 16.7 mm, vias 2 -> 0
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Changed lines of the file:
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@@
 <layer number="27" name="tValues" color="7" fill="1" visible="no" active="yes"/>
 <layer number="28" name="bValues" color="7" fill="1" visible="no" active="yes"/>
-<layer number="29" name="tStop" color="7" fill="3" visible="yes" active="yes"/>
-<layer number="30" name="bStop" color="7" fill="6" visible="yes" active="yes"/>
-<layer number="31" name="tCream" color="7" fill="4" visible="yes" active="yes"/>
-<layer number="32" name="bCream" color="7" fill="5" visible="yes" active="yes"/>
+<layer number="29" name="tStop" color="7" fill="3" visible="no" active="yes"/>
+<layer number="30" name="bStop" color="7" fill="6" visible="no" active="yes"/>
+<layer number="31" name="tCream" color="7" fill="4" visible="no" active="yes"/>
+<layer number="32" name="bCream" color="7" fill="5" visible="no" active="yes"/>
 <layer number="33" name="tFinish" color="6" fill="3" visible="no" active="yes"/>
 <layer number="34" name="bFinish" color="6" fill="6" visible="no" active="yes"/>
@@
 <via x="19.812" y="13.97" extent="1-16" drill="0.381"/>
 </signal>
-<signal name="M1A">
+<signal name="M2A">
 <contactref element="D1" pad="1"/>
 <contactref element="U2" pad="4"/>
@@
 <wire x1="33.054" y1="31.843" x2="33.655" y2="31.242" width="0.508" layer="1"/>
 </signal>
-<signal name="M1B">
+<signal name="M2B">
 <contactref element="U2" pad="5"/>
 <contactref element="D2" pad="1"/>
@@
 <wire x1="36.449" y1="22.733" x2="37.211" y2="23.495" width="0.508" layer="16"/>
 </signal>
-<signal name="M2A">
+<signal name="M1A">
 <contactref element="U2" pad="16"/>
 <contactref element="D3" pad="1"/>
@@
 <wire x1="4.318" y1="43.688" x2="1.397" y2="43.688" width="0.508" layer="1"/>
 </signal>
-<signal name="M2B">
+<signal name="M1B">
 <contactref element="U2" pad="17"/>
 <contactref element="D4" pad="1"/>
@@
 <wire x1="27.52" y1="40.855" x2="28.067" y2="41.402" width="0.1524" layer="1"/>
 </signal>
-<signal name="ENC1B">
+<signal name="ENC2B">
 <contactref element="U1" pad="24"/>
 <wire x1="30.107" y1="35.552" x2="29.5275" y2="36.1315" width="0.1524" layer="1"/>
@@
 <wire x1="30.115" y1="35.56" x2="30.107" y2="35.552" width="0.1524" layer="1"/>
 </signal>
-<signal name="ENC1A">
+<signal name="ENC2A">
 <contactref element="JP6" pad="P$3"/>
 <contactref element="U1" pad="32"/>
@@
 <wire x1="16.383" y1="42.164" x2="17.018" y2="42.164" width="0.1524" layer="1"/>
 </signal>
-<signal name="ENC2B">
+<signal name="ENC1B">
 <contactref element="U1" pad="1"/>
 <contactref element="JP5" pad="P$5"/>
@@
 <wire x1="14.5609" y1="42.3545" x2="14.6304" y2="42.424" width="0.1524" layer="1"/>
 </signal>
-<signal name="ENC2A">
+<signal name="ENC1A">
 <contactref element="U1" pad="23"/>
 <via x="6.604" y="42.418" extent="1-16" drill="0.3302"/>
@@
 <wire x1="5.31435" y1="35.56" x2="5.30635" y2="35.552" width="0.1524" layer="1"/>
 </signal>
-<signal name="M1+">
+<signal name="M2+">
 <contactref element="U2" pad="7"/>
 <contactref element="U1" pad="2"/>
@@
 </signal>
 <signal name="M1-">
-<contactref element="U2" pad="9"/>
-<contactref element="U1" pad="13"/>
-<wire x1="25.908" y1="25.019" x2="24.13" y2="25.019" width="0.254" layer="1"/>
-<wire x1="24.13" y1="25.019" x2="23.4315" y2="25.7175" width="0.254" layer="1"/>
-<wire x1="23.4315" y1="25.7175" x2="23.368" y2="33.147" width="0.254" layer="1"/>
-<wire x1="23.368" y1="33.147" x2="22.987" y2="33.528" width="0.254" layer="1"/>
-<wire x1="19.323" y1="35.3314" x2="19.323" y2="33.89" width="0.254" layer="1"/>
-<wire x1="19.323" y1="33.89" x2="19.685" y2="33.528" width="0.254" layer="1"/>
-<wire x1="19.685" y1="33.528" x2="22.987" y2="33.528" width="0.254" layer="1"/>
-</signal>
-<signal name="M2-">
 <contactref element="U2" pad="15"/>
 <contactref element="U1" pad="12"/>
@@
 <wire x1="17.907" y1="32.258" x2="15.113" y2="32.258" width="0.254" layer="1"/>
 </signal>
-<signal name="M2+">
+<signal name="M1+">
 <contactref element="U2" pad="13"/>
 <contactref element="U1" pad="11"/>
@@
 <wire x1="17.145" y1="33.02" x2="14.351" y2="33.02" width="0.254" layer="1"/>
 </signal>
-<signal name="PWM2">
+<signal name="PWM1">
 <contactref element="U2" pad="14"/>
 <contactref element="U1" pad="9"/>
@@
 <wire x1="14.351" y1="35.3314" x2="15.0622" y2="35.3314" width="0.254" layer="16"/>
 </signal>
-<signal name="PWM1">
+<signal name="PWM2">
 <contactref element="U2" pad="8"/>
 <contactref element="U1" pad="10"/>
@@
 <wire x1="17.526" y1="23.749" x2="24.511" y2="23.749" width="0.254" layer="16"/>
 </signal>
-<signal name="SENSE_2">
+<signal name="SENSE_1">
 <contactref element="U2" pad="19"/>
 <contactref element="R4" pad="2"/>
@@
 <wire x1="20.923" y1="45.346" x2="21.209" y2="45.378" width="0.1524" layer="1"/>
 </signal>
-<signal name="SENSE_1">
+<signal name="SENSE_2">
 <contactref element="R2" pad="2"/>
 <contactref element="R3" pad="2"/>
@@
 <wire x1="15.152" y1="46.1645" x2="15.5965" y2="46.609" width="0.1524" layer="1"/>
 </signal>
+<signal name="M2-">
+<contactref element="U1" pad="13"/>
+<contactref element="U2" pad="9"/>
+<wire x1="25.908" y1="25.019" x2="24.13" y2="25.019" width="0.254" layer="1"/>
+<wire x1="24.13" y1="25.019" x2="23.4315" y2="25.7175" width="0.254" layer="1"/>
+<wire x1="23.4315" y1="25.7175" x2="23.368" y2="33.147" width="0.254" layer="1"/>
+<wire x1="23.368" y1="33.147" x2="22.987" y2="33.528" width="0.254" layer="1"/>
+<wire x1="19.323" y1="33.89" x2="19.685" y2="33.528" width="0.254" layer="1"/>
+<wire x1="19.685" y1="33.528" x2="22.987" y2="33.528" width="0.254" layer="1"/>
+<wire x1="19.323" y1="33.89" x2="19.323" y2="35.3314" width="0.254" layer="1"/>
+</signal>
 </signals>
